File: eagle/rauschsimulator_V4.sch (EAGLE design)
At the start: 79 parts, among them IC1 MAX3232ESE, Q1 BSS123, Q2 BSS123, Q4 BSS123, SW1 SMS_IP67, SW2 SMS_IP67, SW3 SMS_IP67, SW4 SMS_IP67, SW5 SMS_IP67, U1 TSR_1-2450

Commit message: update old/discontinued schematics and layout
Parts:
- removed R24, R25: 3k3, rcl:R-EU_R0603
- removed R26, R27, R28: 56k, rcl:R-EU_R0603
- C1, C2, C3, C4: value 1u/16V -> 200n
Connections:
- removed net N$11: R26.1, U$5.P3
- removed net N$12: C12.1, R24.2, R25.1, U$2.PA0(ADC0/AREF)
- removed net N$37: R27.1, U$4.P3
- removed net N$39: R28.1, U$3.P3
- removed net VCC: C10.1, C11.1, C13.1, C17.+, C9.1, IC1P.VCC, Q1.G, Q2.G, R13.2, R19.2, R21.2, R25.2, R26.2, R27.2, R28.2, R4.2, R5.2, R6.2, U$1.2, U$13.VOUT, U$2.AVCC, U$2.VCC@1, U$2.VCC@2, U$2.VCC@3
- new net N$19: U$2.PC2(OC0C/RXD0)
- new net N$29: U$2.PC3(OC0D/TXD0)
- new net N$30: U$2.PC4(OC1A/!SS!)
- new net N$31: U$2.PC5(OC1B/MOSI/XCK1)
- new net N$32: U$2.PC6(MISO/RXD1)
- new net N$33: U$2.PC7(SCK/TXD1/CLKO/EVO)
- new net N$34: U$2.PD0(OC0A)
- new net VCC_3V: C10.1, C11.1, C12.1, C13.1, C17.+, C9.1, IC1P.VCC, Q1.G, Q2.G, R13.2, R19.2, R21.2, R4.2, R5.2, R6.2, U$1.2, U$13.VOUT, U$2.AVCC, U$2.PA0(ADC0/AREF), U$2.VCC@1, U$2.VCC@2, U$2.VCC@3, U$3.P3, U$4.P3, U$5.P3
- net GND: now also C19.1; no longer C19.2, R24.1
- net VCC_5V: now also C19.2; no longer C19.1
Other:
- note added: "Andere Tasten ( die nicht so sehr prellen !!)"
- note removed: "GATE Widerstand an SUPPLY_CTRL"
- note removed: "an SP49 tatsaechlich VCC_5V benoetigt?"
- moved on the sheet: C12, C19, R4, R5, R6

Commit message: updated schematics to fix ADC ref voltage
Parts:
- added R24, R25: 3k3, rcl:R-EU_R0603
- added R26, R27, R28: 56k, rcl:R-EU_R0603
- C1, C2, C3, C4: value 200n -> 1u/16V
Connections:
- removed net N$19: U$2.PC2(OC0C/RXD0)
- removed net N$29: U$2.PC3(OC0D/TXD0)
- removed net N$30: U$2.PC4(OC1A/!SS!)
- removed net N$31: U$2.PC5(OC1B/MOSI/XCK1)
- removed net N$32: U$2.PC6(MISO/RXD1)
- removed net N$33: U$2.PC7(SCK/TXD1/CLKO/EVO)
- removed net N$34: U$2.PD0(OC0A)
- removed net VCC_3V: C10.1, C11.1, C12.1, C13.1, C17.+, C9.1, IC1P.VCC, Q1.G, Q2.G, R13.2, R19.2, R21.2, R4.2, R5.2, R6.2, U$1.2, U$13.VOUT, U$2.AVCC, U$2.PA0(ADC0/AREF), U$2.VCC@1, U$2.VCC@2, U$2.VCC@3, U$3.P3, U$4.P3, U$5.P3
- new net N$11: R26.1, U$5.P3
- new net N$12: C12.1, R24.2, R25.1, U$2.PA0(ADC0/AREF)
- new net N$37: R27.1, U$4.P3
- new net N$39: R28.1, U$3.P3
- new net VCC: C10.1, C11.1, C13.1, C17.+, C9.1, IC1P.VCC, Q1.G, Q2.G, R13.2, R19.2, R21.2, R25.2, R26.2, R27.2, R28.2, R4.2, R5.2, R6.2, U$1.2, U$13.VOUT, U$2.AVCC, U$2.VCC@1, U$2.VCC@2, U$2.VCC@3
- net GND: now also C19.2, R24.1; no longer C19.1
- net VCC_5V: now also C19.1; no longer C19.2
Other:
- note added: "GATE Widerstand an SUPPLY_CTRL"
- note added: "an SP49 tatsaechlich VCC_5V benoetigt?"
- note removed: "Andere Tasten ( die nicht so sehr prellen !!)"
- moved on the sheet: C12, C19, R4, R5, R6
