File: eagle/rxsms-2.0.brd (EAGLE design)
At the start: 160 x 100 mm, 139 parts, among them Q1 opt, Q10 BSS123, Q11 BSS123, Q12 BSS123, Q2 BSS123, Q3 BSS123, Q4 BSS123, Q5 BSS123, Q6 BSS123, Q7 BSS123, Q8 BSS123, Q9 BSS123, T1 SMS_IP67, T10 SWITCH_LED, T2 SMS_IP67, T3 SWITCH_LED, T4 SMS_IP67, T5 SMS_IP67, T6 SWITCH_LED, T7 SWITCH_LED, T8 SWITCH_LED, T9 SMS_IP67, U1 MAX3232ESE, U2 XMEGA-A4UTQFP, U3 TSR_1-2450, U4 LM1117, U5 TMV_0505EN, U6 ADUM3160, U7 TPS73125, X1 PN61729-S

Commit message: updated switch+led
Changed lines of the file:
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@@
 <contactref element="LED8" pad="C"/>
 <wire x1="-272.05" y1="-736.6" x2="-277.13" y2="-736.6" width="0" layer="19" extent="1-1"/>
-<wire x1="-261.62" y1="-731.52" x2="-272.05" y2="-736.6" width="0" layer="19" extent="1-1"/>
-<wire x1="-261.62" y1="-728.98" x2="-261.62" y2="-731.52" width="0" layer="19" extent="1-1"/>
-<wire x1="-261.62" y1="-720.09" x2="-261.62" y2="-728.98" width="0" layer="19" extent="1-1"/>
-<wire x1="-276.915" y1="-710.78" x2="-261.62" y2="-720.09" width="0" layer="19" extent="1-1"/>
+<wire x1="-256.54" y1="-731.52" x2="-272.05" y2="-736.6" width="0" layer="19" extent="1-1"/>
+<wire x1="-256.54" y1="-728.98" x2="-256.54" y2="-731.52" width="0" layer="19" extent="1-1"/>
+<wire x1="-256.54" y1="-720.09" x2="-256.54" y2="-728.98" width="0" layer="19" extent="1-1"/>
+<wire x1="-276.915" y1="-710.78" x2="-256.54" y2="-720.09" width="0" layer="19" extent="1-1"/>
 <wire x1="-276.915" y1="-696.58" x2="-276.915" y2="-710.78" width="0" layer="19" extent="1-1"/>
-<wire x1="-261.62" y1="-692.15" x2="-276.915" y2="-696.58" width="0" layer="19" extent="1-1"/>
-<wire x1="-261.62" y1="-689.61" x2="-261.62" y2="-692.15" width="0" layer="19" extent="1-1"/>
-<wire x1="-261.62" y1="-680.72" x2="-261.62" y2="-689.61" width="0" layer="19" extent="1-1"/>
-<wire x1="-261.62" y1="-678.18" x2="-261.62" y2="-680.72" width="0" layer="19" extent="1-1"/>
-<wire x1="-273.812" y1="-660.4" x2="-261.62" y2="-678.18" width="0" layer="19" extent="1-1"/>
-<wire x1="-261.62" y1="-765.81" x2="-272.05" y2="-736.6" width="0" layer="19" extent="1-1"/>
-<wire x1="-283.48" y1="-770.89" x2="-261.62" y2="-765.81" width="0" layer="19" extent="1-1"/>
+<wire x1="-256.54" y1="-692.15" x2="-276.915" y2="-696.58" width="0" layer="19" extent="1-1"/>
+<wire x1="-256.54" y1="-689.61" x2="-256.54" y2="-692.15" width="0" layer="19" extent="1-1"/>
+<wire x1="-256.54" y1="-680.72" x2="-256.54" y2="-689.61" width="0" layer="19" extent="1-1"/>
+<wire x1="-256.54" y1="-678.18" x2="-256.54" y2="-680.72" width="0" layer="19" extent="1-1"/>
+<wire x1="-273.812" y1="-660.4" x2="-256.54" y2="-678.18" width="0" layer="19" extent="1-1"/>
+<wire x1="-256.54" y1="-765.81" x2="-272.05" y2="-736.6" width="0" layer="19" extent="1-1"/>
+<wire x1="-283.48" y1="-770.89" x2="-256.54" y2="-765.81" width="0" layer="19" extent="1-1"/>
 <wire x1="-295.91" y1="-770.41" x2="-283.48" y2="-770.89" width="0" layer="19" extent="1-1"/>
 <wire x1="-308.665" y1="-818.5" x2="-295.91" y2="-770.41" width="0" layer="19" extent="1-1"/>
@@
 <contactref element="T3" pad="K"/>
 <wire x1="-124.14" y1="-162.56" x2="-105.41" y2="-129.54" width="0" layer="19" extent="1-1"/>
-<wire x1="-261.62" y1="-717.55" x2="-124.14" y2="-162.56" width="0" layer="19" extent="1-1"/>
-<wire x1="-295.91" y1="-790.73" x2="-261.62" y2="-717.55" width="0" layer="19" extent="1-1"/>
+<wire x1="-256.54" y1="-717.55" x2="-124.14" y2="-162.56" width="0" layer="19" extent="1-1"/>
+<wire x1="-295.91" y1="-790.73" x2="-256.54" y2="-717.55" width="0" layer="19" extent="1-1"/>
 </signal>
 <signal name="!SIM_SODS">
@@
 <contactref element="T10" pad="K"/>
 <wire x1="-124.14" y1="-156.21" x2="-105.41" y2="-116.84" width="0" layer="19" extent="1-1"/>
-<wire x1="-261.62" y1="-763.27" x2="-124.14" y2="-156.21" width="0" layer="19" extent="1-1"/>
-<wire x1="-295.91" y1="-804.7" x2="-261.62" y2="-763.27" width="0" layer="19" extent="1-1"/>
+<wire x1="-256.54" y1="-763.27" x2="-124.14" y2="-156.21" width="0" layer="19" extent="1-1"/>
+<wire x1="-295.91" y1="-804.7" x2="-256.54" y2="-763.27" width="0" layer="19" extent="1-1"/>
 </signal>
 <signal name="EXPPWR_EN">
@@
 <contactref element="T4" pad="3"/>
 <contactref element="T4" pad="4"/>
-<wire x1="-332.685" y1="-831.2" x2="-261.62" y2="-687.07" width="0" layer="19" extent="1-1"/>
+<wire x1="-332.685" y1="-831.2" x2="-256.54" y2="-687.07" width="0" layer="19" extent="1-1"/>
 <wire x1="-332.685" y1="-845.4" x2="-332.685" y2="-831.2" width="0" layer="19" extent="1-1"/>
-<wire x1="-225.74" y1="-447.04" x2="-261.62" y2="-687.07" width="0" layer="19" extent="1-1"/>
+<wire x1="-225.74" y1="-447.04" x2="-256.54" y2="-687.07" width="0" layer="19" extent="1-1"/>
 </signal>
 <signal name="N$37">
@@
 <contactref element="T5" pad="3"/>
 <contactref element="T5" pad="4"/>
-<wire x1="-261.62" y1="-675.64" x2="-225.74" y2="-469.9" width="0" layer="19" extent="1-1"/>
-<wire x1="-319.985" y1="-831.2" x2="-261.62" y2="-675.64" width="0" layer="19" extent="1-1"/>
+<wire x1="-256.54" y1="-675.64" x2="-225.74" y2="-469.9" width="0" layer="19" extent="1-1"/>
+<wire x1="-319.985" y1="-831.2" x2="-256.54" y2="-675.64" width="0" layer="19" extent="1-1"/>
 <wire x1="-319.985" y1="-845.4" x2="-319.985" y2="-831.2" width="0" layer="19" extent="1-1"/>
 </signal>
@@
 <contactref element="T1" pad="3"/>
 <contactref element="T1" pad="4"/>
-<wire x1="-290.51" y1="-737.87" x2="-261.62" y2="-726.44" width="0" layer="19" extent="1-1"/>
+<wire x1="-290.51" y1="-737.87" x2="-256.54" y2="-726.44" width="0" layer="19" extent="1-1"/>
 <wire x1="-345.385" y1="-831.2" x2="-290.51" y2="-737.87" width="0" layer="19" extent="1-1"/>
 <wire x1="-345.385" y1="-845.4" x2="-345.385" y2="-831.2" width="0" layer="19" extent="1-1"/>
@@
 <contactref element="T2" pad="4"/>
 <contactref element="T3" pad="A1"/>
-<wire x1="-261.62" y1="-715.01" x2="-269.185" y2="-710.78" width="0" layer="19" extent="1-1"/>
+<wire x1="-256.54" y1="-715.01" x2="-269.185" y2="-710.78" width="0" layer="19" extent="1-1"/>
 <wire x1="-269.185" y1="-696.58" x2="-269.185" y2="-710.78" width="0" layer="19" extent="1-1"/>
 <wire x1="-284.16" y1="-737.87" x2="-269.185" y2="-710.78" width="0" layer="19" extent="1-1"/>
@@
 <wire x1="-300.935" y1="-818.5" x2="-300.935" y2="-832.7" width="0" layer="19" extent="1-1"/>
 <wire x1="-290.51" y1="-772.16" x2="-300.935" y2="-818.5" width="0" layer="19" extent="1-1"/>
-<wire x1="-261.62" y1="-760.73" x2="-290.51" y2="-772.16" width="0" layer="19" extent="1-1"/>
+<wire x1="-256.54" y1="-760.73" x2="-290.51" y2="-772.16" width="0" layer="19" extent="1-1"/>
 </signal>
 <signal name="SW_LO">
@@
 <contactref element="T8" pad="A"/>
 <contactref element="R36" pad="2"/>
-<wire x1="-294.96" y1="-778.51" x2="-259.08" y2="-728.98" width="0" layer="19" extent="1-1"/>
+<wire x1="-294.96" y1="-778.51" x2="-254" y2="-728.98" width="0" layer="19" extent="1-1"/>
 </signal>
 <signal name="LED_LO">
@@
 <contactref element="T7" pad="A"/>
 <contactref element="R42" pad="2"/>
-<wire x1="-307.66" y1="-838.2" x2="-259.08" y2="-678.18" width="0" layer="19" extent="1-1"/>
+<wire x1="-307.66" y1="-838.2" x2="-254" y2="-678.18" width="0" layer="19" extent="1-1"/>
 </signal>
 <signal name="LED_ERRINH">
@@
 <contactref element="R45" pad="2"/>
 <contactref element="T6" pad="A"/>
-<wire x1="-259.08" y1="-689.61" x2="-358.46" y2="-857.25" width="0" layer="19" extent="1-1"/>
+<wire x1="-254" y1="-689.61" x2="-358.46" y2="-857.25" width="0" layer="19" extent="1-1"/>
 </signal>
 <signal name="LED_TO_EXP_ACTIVE">

Commit message: progress on schematics
  * add of TVS supressor diodes for USB
  * add of RC-filter for USB
  * new library for light pipe
  * add of light-pipe to the schematics
  * add of pinheaders for two reserved UARTs
  * some resistors for LEDs updated, not final yet
  * some OC_FARNELL order codes added
  * assignment of signals to uC symbol
  * implement current sense functionality
Parts:
- added C34: 4n7, rcl:C0805K
- added JP3, JP4: (no value), pinhead:1X04
- added R48: 1M, rcl:R0805
- added R49: 220, rcl:R0805
- added R50: 330, rcl:R0805
- added U8: NUP2202W1, nup2202w1:SOT363_PHILIPS
- added X5: RLP2-200-500, light-pipe:RLP2-200-500
- LED1, LED2, LED3: value (none) -> YELLOW
- LED4, LED5, LED8: value (none) -> GREEN
- LED6, LED7: value (none) -> BERNSTEIN
- R36, R37, R38, R39, R40, R41, R42, R45, R46, R47: value 220 -> 68
- moved R27 438.3 mm to (-284.5, -129.5)
- moved R33 438.3 mm to (-284.5, -193.0)
- moved SJ2 438.3 mm to (-283.2, -217.2)
- moved C22 438.3 mm to (-222.2, 82.5)
- moved C25 438.3 mm to (-288.3, -298.4)
- moved C26 438.3 mm to (-283.2, -298.4)
- moved C28 438.3 mm to (-229.9, -8.89)
- moved C32 438.3 mm to (-234.9, -48.3)
- moved C33 438.3 mm to (-234.9, -61.0)
- moved LED4 438.3 mm to (-325.1, -400.1)
- moved LED6 438.3 mm to (-375.9, -425.4)
- moved LED8 438.3 mm to (-388.6, -431.8)
- moved OK2 438.3 mm to (-271.8, -106.7)
- moved OK3 438.3 mm to (-281.9, -121.9)
- moved OK4 438.3 mm to (-281.9, -170.2)
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Connections:
- removed net N$15 (its old number): C17.2, C18.2, U6.2, U6.8, X1.4, X1.S1, X1.S2
- removed net N$17 (its old number): C18.1, U6.1, X1.1
- removed net USB-D+: R15.1
- removed net USB_D-: R14.1
- new net ADC_CURRENT_SENSE: R50.2, U$6.PIN4, U2.43
- new net N$68: R13.2, U8.1, X1.3
- new net RESERVED_UART0_RX: JP4.2, U2.12
- new net RESERVED_UART0_TX: JP4.3, U2.13
- new net RESERVED_UART1_RX: JP3.2, U2.16
- new net RESERVED_UART1_TX: JP3.3, U2.17
- new net USB_GND: C17.2, C18.2, C34.1, R48.2, U6.2, U6.8, X1.4
- new net USB_SHIELD: C34.2, R48.1, U8.2, X1.S1, X1.S2
- new net USB_VBUS: C18.1, U6.1, U8.5, X1.1
- net !SIM_LO: now also U2.24
- net !SIM_SODS: now also U2.28
- net !SIM_SOE: now also U2.25
- net +3V3: now also JP3.1, JP4.1; no longer LED8.A
- net +5V: now also R49.2
- net ADC_POTI_BIT_ERROR_RATE: now also U2.40
- net ADC_POTI_DROP_DURATION: now also U2.42
- net ADC_POTI_DROP_RATE: now also U2.41
- net ADC_REF: now also U2.4
- net DEBUG_RX_D-: now also R14.1, U2.26
- net DEBUG_TX_D+: now also R15.1, U2.27
- net EXPPWR_EN: now also U2.29
- net GND: now also JP3.4, JP4.4, R50.1
- net LED_ERRINH: now also U2.15
- net LED_LO: now also U2.14
- net LED_TO_EXP_ACTIVE: now also U2.10
- net LED_TO_GND_ACTIVE: now also U2.11
- net N$23: now also LED8.A, R49.1; no longer R13.2, X1.3
- net N$24: now also U8.6
- net SW_ERRINH: now also U2.3
- net SW_LO: now also U2.5
- net SW_PWR: now also U2.2
- net SW_SODS: now also U2.7
- net SW_SOE: now also U2.6
- net UART_EXP_RX: now also U2.22
- net UART_EXP_TX: now also U2.23
- net UART_GND_RX: now also U2.32
- net UART_GND_TX: now also U2.33

Commit message: reordered signals on uC
Connections:
- net !SIM_LO: no longer U2.24
- net !SIM_SODS: no longer U2.28
- net !SIM_SOE: no longer U2.25
- net DEBUG_RX_D-: no longer U2.26
- net DEBUG_TX_D+: no longer U2.27
- net EXPPWR_EN: no longer U2.29
- net LED_ERRINH: no longer U2.15
- net LED_LO: no longer U2.14
- net LED_TO_EXP_ACTIVE: no longer U2.10
- net LED_TO_GND_ACTIVE: no longer U2.11
- net RESERVED_UART0_RX: no longer U2.12
- net RESERVED_UART0_TX: no longer U2.13
- net RESERVED_UART1_RX: no longer U2.16
- net RESERVED_UART1_TX: no longer U2.17
- net SW_ERRINH: no longer U2.3
- net SW_LO: now also U2.7; no longer U2.5
- net SW_PWR: no longer U2.2
- net SW_SODS: now also U2.5; no longer U2.7
- net UART_EXP_RX: no longer U2.22
- net UART_EXP_TX: no longer U2.23
- net UART_GND_RX: no longer U2.32
- net UART_GND_TX: no longer U2.33
Changed lines of the file:
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@@
 <contactref element="U$4" pad="19"/>
 <contactref element="R4" pad="1"/>
-<contactref element="U2" pad="24"/>
 <wire x1="-124.14" y1="-168.91" x2="-105.41" y2="-132.08" width="0" layer="19" extent="1-1"/>
-<wire x1="-93.43" y1="26.06" x2="-105.41" y2="-132.08" width="0" layer="19" extent="1-1"/>
 </signal>
 <signal name="!SIM_SOE">
@@
 <contactref element="T3" pad="K"/>
 <contactref element="LED2" pad="C"/>
-<contactref element="U2" pad="25"/>
 <wire x1="-124.14" y1="-162.56" x2="-105.41" y2="-129.54" width="0" layer="19" extent="1-1"/>
-<wire x1="-93.43" y1="25.26" x2="-105.41" y2="-129.54" width="0" layer="19" extent="1-1"/>
 <wire x1="-266.7" y1="-279.4" x2="-124.14" y2="-162.56" width="0" layer="19" extent="1-1"/>
 <wire x1="-401.32" y1="-449.1" x2="-266.7" y2="-279.4" width="0" layer="19" extent="1-1"/>
@@
 <contactref element="T10" pad="K"/>
 <contactref element="LED3" pad="C"/>
-<contactref element="U2" pad="28"/>
 <wire x1="-124.14" y1="-156.21" x2="-105.41" y2="-116.84" width="0" layer="19" extent="1-1"/>
-<wire x1="-93.43" y1="22.86" x2="-105.41" y2="-116.84" width="0" layer="19" extent="1-1"/>
 <wire x1="-266.7" y1="-325.12" x2="-124.14" y2="-156.21" width="0" layer="19" extent="1-1"/>
 <wire x1="-407.67" y1="-449.1" x2="-266.7" y2="-325.12" width="0" layer="19" extent="1-1"/>
@@
 <contactref element="R44" pad="1"/>
 <contactref element="R45" pad="1"/>
-<contactref element="U2" pad="29"/>
-<wire x1="-370.52" y1="-412.75" x2="-370.52" y2="-419.1" width="0" layer="19" extent="1-1"/>
-<wire x1="-129.86" y1="-175.26" x2="-370.52" y2="-412.75" width="0" layer="19" extent="1-1"/>
 <wire x1="-112.71" y1="-149.69" x2="-129.86" y2="-175.26" width="0" layer="19" extent="1-1"/>
-<wire x1="-93.43" y1="22.06" x2="-112.71" y2="-149.69" width="0" layer="19" extent="1-1"/>
+<wire x1="-370.52" y1="-412.75" x2="-129.86" y2="-175.26" width="0" layer="19" extent="1-1"/>
+<wire x1="-370.52" y1="-419.1" x2="-370.52" y2="-412.75" width="0" layer="19" extent="1-1"/>
 </signal>
 <signal name="N$16">
@@
 <contactref element="R8" pad="1"/>
 <contactref element="JP1" pad="1"/>
-<contactref element="U2" pad="22"/>
-<wire x1="-131.76" y1="-208.28" x2="-290.83" y2="-220.98" width="0" layer="19" extent="1-1"/>
 <wire x1="-128.59" y1="-201.76" x2="-131.76" y2="-208.28" width="0" layer="19" extent="1-1"/>
-<wire x1="-91.63" y1="28.66" x2="-128.59" y2="-201.76" width="0" layer="19" extent="1-1"/>
+<wire x1="-290.83" y1="-220.98" x2="-131.76" y2="-208.28" width="0" layer="19" extent="1-1"/>
 </signal>
 <signal name="N$21">
@@
 <contactref element="R10" pad="1"/>
 <contactref element="JP2" pad="2"/>
-<contactref element="U2" pad="23"/>
-<wire x1="-131.76" y1="-229.87" x2="-298.45" y2="-218.44" width="0" layer="19" extent="1-1"/>
 <wire x1="-128.59" y1="-223.35" x2="-131.76" y2="-229.87" width="0" layer="19" extent="1-1"/>
-<wire x1="-93.43" y1="26.86" x2="-128.59" y2="-223.35" width="0" layer="19" extent="1-1"/>
+<wire x1="-298.45" y1="-218.44" x2="-131.76" y2="-229.87" width="0" layer="19" extent="1-1"/>
 </signal>
 <signal name="EXP_CHG_IN">
@@
 <contactref element="C28" pad="1"/>
 <contactref element="R19" pad="2"/>
-<contactref element="U2" pad="2"/>
 <wire x1="-230.87" y1="-8.89" x2="-234" y2="-8.89" width="0" layer="19" extent="1-1"/>
-<wire x1="-81.83" y1="19.66" x2="-230.87" y2="-8.89" width="0" layer="19" extent="1-1"/>
 </signal>
 <signal name="N$35">
@@
 <contactref element="C29" pad="1"/>
 <contactref element="R20" pad="2"/>
-<contactref element="U2" pad="3"/>
 <wire x1="-230.87" y1="-31.75" x2="-234" y2="-31.75" width="0" layer="19" extent="1-1"/>
-<wire x1="-81.83" y1="20.46" x2="-230.87" y2="-31.75" width="0" layer="19" extent="1-1"/>
 </signal>
 <signal name="ADC_REF">
@@
 <signal name="UART_GND_TX">
 <contactref element="Q6" pad="1"/>
-<contactref element="U2" pad="33"/>
-<wire x1="-275.27" y1="-76.03" x2="-93.43" y2="18.86" width="0" layer="19" extent="1-1"/>
 </signal>
 <signal name="N$39">
@@
 <contactref element="R27" pad="1"/>
 <contactref element="OK3" pad="6"/>
-<contactref element="U2" pad="32"/>
 <wire x1="-281.305" y1="-118.8466" x2="-285.43" y2="-129.54" width="0" layer="19" extent="1-1"/>
-<wire x1="-93.43" y1="19.66" x2="-281.305" y2="-118.8466" width="0" layer="19" extent="1-1"/>
 </signal>
 <signal name="N$47">
@@
 <contactref element="R35" pad="1"/>
 <contactref element="R15" pad="1"/>
-<contactref element="U2" pad="27"/>
-<wire x1="-93.43" y1="23.66" x2="-180.02" y2="140.97" width="0" layer="19" extent="1-1"/>
-<wire x1="-285.43" y1="-205.74" x2="-180.02" y2="140.97" width="0" layer="19" extent="1-1"/>
+<wire x1="-180.02" y1="140.97" x2="-285.43" y2="-205.74" width="0" layer="19" extent="1-1"/>
 </signal>
 <signal name="DEBUG_RX_D-">
 <contactref element="R33" pad="1"/>
 <contactref element="R14" pad="1"/>
-<contactref element="U2" pad="26"/>
-<wire x1="-93.43" y1="24.46" x2="-180.02" y2="147.32" width="0" layer="19" extent="1-1"/>
-<wire x1="-285.43" y1="-193.04" x2="-180.02" y2="147.32" width="0" layer="19" extent="1-1"/>
+<wire x1="-180.02" y1="147.32" x2="-285.43" y2="-193.04" width="0" layer="19" extent="1-1"/>
 </signal>
 <signal name="N$26">
@@
 <contactref element="C25" pad="1"/>
 <contactref element="R16" pad="2"/>
-<contactref element="U2" pad="5"/>
-<wire x1="-298.77" y1="-299.72" x2="-289.29" y2="-298.45" width="0" layer="19" extent="1-1"/>
-<wire x1="-81.83" y1="22.06" x2="-289.29" y2="-298.45" width="0" layer="19" extent="1-1"/>
+<contactref element="U2" pad="7"/>
+<wire x1="-289.29" y1="-298.45" x2="-298.77" y2="-299.72" width="0" layer="19" extent="1-1"/>
+<wire x1="-81.83" y1="23.66" x2="-289.29" y2="-298.45" width="0" layer="19" extent="1-1"/>
 </signal>
 <signal name="SW_SOE">
@@
 <contactref element="C27" pad="1"/>
 <contactref element="R18" pad="2"/>
-<contactref element="U2" pad="7"/>
-<wire x1="-295.64" y1="-332.74" x2="-81.83" y2="23.66" width="0" layer="19" extent="1-1"/>
-<wire x1="-298.77" y1="-334.01" x2="-295.64" y2="-332.74" width="0" layer="19" extent="1-1"/>
+<contactref element="U2" pad="5"/>
+<wire x1="-295.64" y1="-332.74" x2="-298.77" y2="-334.01" width="0" layer="19" extent="1-1"/>
+<wire x1="-81.83" y1="22.06" x2="-295.64" y2="-332.74" width="0" layer="19" extent="1-1"/>
 </signal>
 <signal name="N$31">
@@
 <contactref element="R37" pad="1"/>
 <contactref element="R36" pad="1"/>
-<contactref element="U2" pad="14"/>
 <wire x1="-307.02" y1="-340.36" x2="-307.02" y2="-346.71" width="0" layer="19" extent="1-1"/>
-<wire x1="-85.23" y1="28.66" x2="-307.02" y2="-340.36" width="0" layer="19" extent="1-1"/>
 </signal>
 <signal name="N$34">
@@
 <contactref element="R43" pad="1"/>
 <contactref element="R42" pad="1"/>
-<contactref element="U2" pad="15"/>
 <wire x1="-319.72" y1="-400.05" x2="-326.07" y2="-406.4" width="0" layer="19" extent="1-1"/>
-<wire x1="-86.03" y1="28.66" x2="-326.07" y2="-406.4" width="0" layer="19" extent="1-1"/>
 </signal>
 <signal name="N$63">
@@
 <signal name="LED_TO_EXP_ACTIVE">
 <contactref element="R46" pad="2"/>
-<contactref element="U2" pad="10"/>
-<wire x1="-81.83" y1="26.06" x2="-368.62" y2="-425.45" width="0" layer="19" extent="1-1"/>
 </signal>
 <signal name="LED_TO_GND_ACTIVE">
 <contactref element="R47" pad="2"/>
-<contactref element="U2" pad="11"/>
-<wire x1="-81.83" y1="26.86" x2="-374.97" y2="-431.8" width="0" layer="19" extent="1-1"/>
 </signal>
 <signal name="N$65">
@@
 <signal name="RESERVED_UART0_RX">
 <contactref element="JP4" pad="2"/>
-<contactref element="U2" pad="12"/>
-<wire x1="-83.63" y1="28.66" x2="-421.64" y2="-477.52" width="0" layer="19" extent="1-1"/>
 </signal>
 <signal name="RESERVED_UART0_TX">
 <contactref element="JP4" pad="3"/>
-<contactref element="U2" pad="13"/>
-<wire x1="-419.1" y1="-477.52" x2="-84.43" y2="28.66" width="0" layer="19" extent="1-1"/>
 </signal>
 <signal name="RESERVED_UART1_RX">
 <contactref element="JP3" pad="2"/>
-<contactref element="U2" pad="16"/>
-<wire x1="-421.64" y1="-471.17" x2="-86.83" y2="28.66" width="0" layer="19" extent="1-1"/>
 </signal>
 <signal name="RESERVED_UART1_TX">
 <contactref element="JP3" pad="3"/>
-<contactref element="U2" pad="17"/>
-<wire x1="-419.1" y1="-471.17" x2="-87.63" y2="28.66" width="0" layer="19" extent="1-1"/>
 </signal>
 </signals>
