File: eagle/rxsms-2.0.brd (EAGLE design)
At the start: 160 x 100 mm, 159 parts, among them Q1 opt, Q10 BSS123, Q11 BSS123, Q12 BSS123, Q2 BSS123, Q3 BSS123, Q4 BSS123, Q5 BSS123, Q6 BSS123, Q7 BSS123, Q8 BSS123, Q9 BSS123, T1 SMS_IP67, T10 SWITCH_LED, T2 SMS_IP67, T3 SWITCH_LED, T4 SMS_IP67, T5 SMS_IP67, T6 SWITCH_LED, T7 SWITCH_LED, T8 SWITCH_LED, T9 SMS_IP67, U1 MAX3232ESE, U2 XMEGA-A4UTQFP, U3 TSR_1-2450, U4 LM1117, U6 ADUM3160, U7 TPS73125, U8 NUP2202W1, X1 PN61729-S, X5 RLP2-200-500

Commit message: Placement of components acording to mechanical CAD
Parts:
- removed LED1, LED2, LED3: YELLOW, led:CHIPLED_1206
- removed LED4, LED5: GREEN, led:CHIPLED_1206
- removed T1, T2, T4, T5, T9: SMS_IP67, SMSIp67:IP67
- removed T10, T3, T6, T7, T8: SWITCH_LED, mentor-switch:SWITCH_LED
- removed U$9: (no value), poti:VERT_POTI
- removed X2, X3: (no value), con-subd:F09HP
- added LED1_LO, LED2_SOE, LED3_SODS: YELLOW, led:CHIPLED_1206
- added LED4_ERRINH, LED5_PWR: GREEN, led:CHIPLED_1206
- added T10_SODS, T3_SOE, T6_PWR, T7_ERRINH, T8_LO: SWITCH_LED, mentor-switch:SWITCH_LED
- added T1_LO, T2_SOE, T4_PWR, T5_ERRINH, T9_SODS: SMS_IP67, SMSIp67:IP67
- added U$7_BER, U$8_DROPR, U$9_DROPDUR: (no value), poti:VERT_POTI
- added X2_GROUNDSTATION, X3_DEBUG: (no value), con-subd:F09HP
- U$7, U$8: device poti:VERT_POTI -> holes:3,2
- moved SJ4 822.6 mm to (144.8, 3.81)
- moved U$12 813.4 mm to (64.8, 85.1), turned to 180 degrees
- moved X6 811.4 mm to (96.5, 113.0)
- moved X5 792.8 mm to (146.2, 105.0), turned to 90 degrees
- moved U$11 786.4 mm to (64.8, 71.1), turned to 180 degrees
- moved LED7 777.6 mm to (146.2, 107.5), turned to 270 degrees
- moved U$10 771.1 mm to (77.5, 66.0), turned to 90 degrees
- moved SV1 764.7 mm to (55.0, 103.1)
- moved R47 750.1 mm to (139.7, 113.0), turned to 180 degrees
- moved R49 747.3 mm to (92.7, 97.8)
- moved LED6 742.5 mm to (146.2, 102.5), turned to 270 degrees
- moved R46 731.1 mm to (139.7, 99.1), turned to 180 degrees
- moved LED8 718.5 mm to (92.7, 101.6)
- moved R48 699.6 mm to (141.0, 6.35)
- moved R50 698.9 mm to (100.3, 16.5), turned to 180 degrees
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Connections:
- net !SIM_LO: now also U2.20
- net !SIM_SODS: now also LED3_SODS.C, T10_SODS.K, U2.24; no longer LED3.C, T10.K
- net !SIM_SOE: now also LED2_SOE.C, T3_SOE.K, U2.21; no longer LED2.C, T3.K
- net ADC_POTI_BIT_ERROR_RATE: now also U$7_BER.P2; no longer U$7.P2
- net ADC_POTI_DROP_DURATION: now also U$9_DROPDUR.P2; no longer U$9.P2
- net ADC_POTI_DROP_RATE: now also U$8_DROPR.P2; no longer U$8.P2
- net ADC_REF: now also U$7_BER.P3, U$8_DROPR.P3, U$9_DROPDUR.P3; no longer U$7.P3, U$8.P3, U$9.P3
- net DEBUG_RX_D-: now also U2.26
- net DEBUG_TX_D+: now also U2.27
- net EXPPWR_EN: now also U2.25
- net EXP_CHG_IN: now also X3_DEBUG.1, X3_DEBUG.6, X3_DEBUG.7; no longer X3.1, X3.6, X3.7
- net EXP_CHG_RET: now also X3_DEBUG.4, X3_DEBUG.8, X3_DEBUG.9; no longer X3.4, X3.8, X3.9
- net GND: now also LED1_LO.C, LED4_ERRINH.C, LED5_PWR.C, T10_SODS.3A, T1_LO.1, T1_LO.2, T2_SOE.1, T2_SOE.2, T3_SOE.3A, T4_PWR.1, T4_PWR.2, T5_ERRINH.1, T5_ERRINH.2, T6_PWR.3A, T6_PWR.K, T7_ERRINH.3A, T7_ERRINH.K, T8_LO.3A, T8_LO.K, T9_SODS.1, T9_SODS.2, U$7_BER.P1, U$8_DROPR.P1, U$9_DROPDUR.P1; no longer LED1.C, LED4.C, LED5.C, T1.1, T1.2, T10.3A, T2.1, T2.2, T3.3A, T4.1, T4.2, T5.1, T5.2, T6.3A, T6.K, T7.3A, T7.K, T8.3A, T8.K, T9.1, T9.2, U$7.P1, U$8.P1, U$9.P1
- net LED_ERRINH: now also U2.10
- net LED_LO: now also U2.11
- net LED_TO_EXP_ACTIVE: now also U2.14
- net LED_TO_GND_ACTIVE: now also U2.15
- net N$10: now also X3_DEBUG.3; no longer X3.3
- net N$15: now also LED2_SOE.A; no longer LED2.A
- net N$17: now also LED3_SODS.A; no longer LED3.A
- net N$26: now also T1_LO.3, T1_LO.4, T8_LO.A1; no longer T1.3, T1.4, T8.A1
- net N$27: now also T2_SOE.3, T2_SOE.4, T3_SOE.A1; no longer T2.3, T2.4, T3.A1
- net N$28: now also T10_SODS.A1, T9_SODS.3, T9_SODS.4; no longer T10.A1, T9.3, T9.4
- net N$3: now also X2_GROUNDSTATION.2; no longer X2.2
- net N$31: now also LED1_LO.A; no longer LED1.A
- net N$32: now also T8_LO.A; no longer T8.A
- net N$34: now also T3_SOE.A
- net N$35: now also T4_PWR.3, T4_PWR.4, T6_PWR.A1; no longer T4.3, T4.4, T6.A1
- net N$37: now also T5_ERRINH.3, T5_ERRINH.4, T7_ERRINH.A1; no longer T5.3, T5.4, T7.A1
- net N$56: now also X2_GROUNDSTATION.G2; no longer X2.G2
- net N$57: now also X3_DEBUG.G2; no longer X3.G2
- net N$61: now also LED4_ERRINH.A; no longer LED4.A
- net N$62: now also T7_ERRINH.A; no longer T7.A
- net N$63: now also LED5_PWR.A; no longer LED5.A
- net N$64: now also T6_PWR.A; no longer T6.A
- net N$8: now also X2_GROUNDSTATION.3; no longer X2.3
- net N$9: now also X3_DEBUG.2; no longer X3.2
- net RESERVED_UART0_RX: now also U2.16
- net RESERVED_UART0_TX: now also U2.17
- net RESERVED_UART1_RX: now also U2.32
- net RESERVED_UART1_TX: now also U2.33
- net SW_ERRINH: now also U2.2
- net SW_PWR: now also U2.3
- net UART_EXP_RX: now also U2.12
- net UART_EXP_TX: now also U2.13
- net UART_GND_RX: now also U2.22
- net UART_GND_TX: now also U2.23
- net VSS: now also X2_GROUNDSTATION.5, X3_DEBUG.5; no longer X2.5, X3.5
Other:
- board size 160 x 100 mm -> 159 x 120.5 mm

Commit message: continued layout
Parts:
- added C40: 100n, rcl:C0805K
- added D1: 3V, diode:SOT23
- added U5: NC7WZ17P6X, NC7WZ17:SOT65P210X110-6N
- R4: value 10k -> 22k
- moved C28 372.5 mm to (138.4, 47.0)
- moved R19 341.7 mm to (106.7, -14.0), turned to 180 degrees
- moved JP2 324.9 mm to (55.9, -6.35)
- moved JP1 319.9 mm to (58.4, -6.35), turned to 180 degrees
- moved C30 313.1 mm to (76.2, 97.8)
- moved R27 312.8 mm to (61.0, 19.7), turned to 90 degrees
- moved R35 304.9 mm to (52.1, -11.4), turned to 180 degrees
- moved R34 304.7 mm to (52.1, -7.62), turned to 180 degrees
- moved R15 304.5 mm to (96.5, 11.4)
- moved OK3 304.5 mm to (54.6, 19.1), turned to 270 degrees
- moved R33 303.7 mm to (52.1, -16.5), turned to 180 degrees
- moved R14 301.0 mm to (91.4, 15.2)
- moved SJ3 299.9 mm to (16.5, 80.0), turned to 90 degrees
- moved R29 298.9 mm to (47.0, 22.9), turned to 90 degrees
- moved Q9 297.3 mm to (47.0, 18.4), turned to 270 degrees
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Connections:
- removed net N$69: SV1.11, SV1.13, SV1.3, SV1.5, SV1.7, SV1.9
- removed net N$71: SJ4.2, X1.S1, X1.S2
- removed net N$72: C34.2, R48.1, SJ4.1
- new net N$73: C40.1, U5.5
- net !EXP_LO: now also SV1.2, U$4.15; no longer U$4.16
- net !EXP_SODS: now also U$4.17; no longer U$4.15
- net !EXP_SOE: now also U$4.16; no longer U$4.17
- net !SIM_LO: now also D1.3, SV1.1, U5.1; no longer U$4.19
- net !SIM_SODS: now also R3.1, U$4.18; no longer R2.1, U$4.13
- net !SIM_SOE: now also R2.1, U$4.19; no longer R3.1, U$4.18
- net ADC_REF: now also JP5.2
- net GND: now also C40.2, D1.1, SV1.10, SV1.11, SV1.12, SV1.13, SV1.14, SV1.3, SV1.4, SV1.5, SV1.6, SV1.7, SV1.8, SV1.9, U5.2
- net N$56: now also X2_GROUNDSTATION.G1; no longer X2_GROUNDSTATION.G2
- net N$57: now also SJ2.1; no longer SJ2.2
- net N$58: now also X4.G1; no longer X4.G2
- net N$60: now also T10_SODS.A
- net N$67: now also U$4.13, U5.6; no longer SV1.10, SV1.12, SV1.14, SV1.4, SV1.6, SV1.8
- net RESERVED_ADC_0: now also JP5.3
- net RESERVED_ADC_1: now also JP5.4
- net USB_GND: now also SJ4.1
- net USB_SHIELD: now also C34.2, R48.1, SJ4.2, X1.S1, X1.S2
- net VSS: now also SJ2.2; no longer SJ2.1
Routing:
- net USB_VBUS: track 0.00 -> 63.5 mm, vias 0 -> 2
- net USB_SHIELD: track 0.00 -> 62.7 mm, vias 0 -> 2
- net !EXP_LO: track 0.00 -> 61.7 mm
- net N$3: track 0.00 -> 48.4 mm
- net +3V3: track 0.00 -> 37.6 mm
- net USB_GND: track 0.00 -> 35.3 mm, vias 0 -> 5
- net N$8: track 0.00 -> 33.2 mm
- net GND: track 0.00 -> 32.9 mm
- net N$68: track 0.00 -> 29.3 mm
- net !EXP_SOE: track 0.00 -> 28.2 mm
- net VDD: track 0.00 -> 25.9 mm
- net !EXP_SODS: track 0.00 -> 24.6 mm
- net N$24: track 0.00 -> 24.3 mm
- net EXP_SERIAL_FROM_EXP-: track 0.00 -> 20.9 mm
- net EXP_SERIAL_FROM_EXP+: track 0.00 -> 20.8 mm, vias 0 -> 1
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- added copper zone on layer 1, net +28V_EXP
- added copper zone on layer 16, net +28V_EXP
- added copper zone on layer 1, net +28V_SUPPLY
- added copper zone on layer 16, net GND
- added copper zone on layer 1, net USB_GND
- added copper zone on layer 16, net USB_GND

Commit message: charging line and some extension headers added
Parts:
- moved JP3 152.7 mm to (69.8, 19.1), turned to 90 degrees
- moved JP6 145.7 mm to (66.0, 19.1), turned to 90 degrees
- moved JP5 139.7 mm to (63.5, 50.8)
- moved JP4 123.4 mm to (45.7, 38.1), turned to 270 degrees
- moved R9 103.6 mm to (48.3, 71.1)
- moved R8 94.0 mm to (43.2, 63.5)
- moved R10 90.9 mm to (29.2, 64.8), turned to 180 degrees
- moved Q4 88.4 mm to (29.2, 69.8)
- moved R11 85.5 mm to (24.1, 71.1), turned to 180 degrees
- moved C9 0.64 mm to (64.1, 26.7)
Routing:
- net RESERVED_UART1_RX: track 0.00 -> 16.4 mm
- net RESERVED_UART1_TX: track 0.00 -> 16.3 mm
- net N$33: track 0.00 -> 15.4 mm
- net N$36: track 0.00 -> 12.5 mm
- net +3V3: track 37.6 -> 48.9 mm
- net GND: track 32.9 -> 43.0 mm
- added copper zone on layer 1, net EXP_CHG_IN
- added copper zone on layer 16, net EXP_CHG_IN
- added copper zone on layer 1, net EXP_CHG_RET

Commit message: most of buttons connected
Parts:
- moved R20 216.5 mm to (124.5, 20.3), turned to 180 degrees
- moved C29 212.5 mm to (124.5, 17.8)
- moved C21 211.1 mm to (105.4, 43.2), turned to 180 degrees
- moved C22 210.4 mm to (100.3, 87.6), turned to 90 degrees
- moved C23 205.9 mm to (101.0, 57.1), turned to 90 degrees
- moved C24 203.9 mm to (101.0, 27.3), turned to 90 degrees
- moved U7 196.9 mm to (104.1, 39.4)
- moved C19 192.8 mm to (104.1, 7.62), turned to 270 degrees
- moved C20 188.0 mm to (101.6, 7.62), turned to 270 degrees
- moved C39 181.5 mm to (100.3, 41.9), turned to 270 degrees
- moved C38 179.0 mm to (100.3, 38.1), turned to 90 degrees
- moved C31 165.9 mm to (83.8, 82.5)
- moved C36 165.5 mm to (85.1, 57.1)
- moved C37 164.7 mm to (85.1, 49.5)
- moved C35 156.9 mm to (71.1, 85.1)
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Routing:
- net GND: track 43.0 -> 231.3 mm, vias 0 -> 2
- net +3V3: track 48.9 -> 111.7 mm
- net N$16: track 0.00 -> 41.2 mm
- net ADC_CURRENT_SENSE: track 0.00 -> 35.1 mm
- net N$27: track 0.00 -> 20.7 mm
- net N$26: track 0.00 -> 20.6 mm
- net N$28: track 0.00 -> 20.5 mm
- net +5V: track 3.67 -> 22.9 mm
- net N$21: track 0.00 -> 15.2 mm
- net N$67: track 0.00 -> 12.7 mm
- net !SIM_SODS: track 0.00 -> 12.0 mm
- net N$66: track 0.00 -> 11.0 mm
- net EXPPWR_EN: track 0.00 -> 10.7 mm
- net ADC_REF: track 0.00 -> 9.49 mm
- net !SIM_LO: track 0.00 -> 8.37 mm
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
Commit message: continued layout
Parts:
- moved R23 66.4 mm to (34.9, 33.0)
- moved R28 63.5 mm to (39.4, 40.6), turned to 0 degrees
- moved R29 62.5 mm to (44.5, 39.4)
- moved Q10 62.3 mm to (35.6, 37.5)
- moved Q9 62.3 mm to (40.6, 37.5)
- moved OK1 57.1 mm to (36.8, 25.4), turned to 0 degrees
- moved OK3 52.9 mm to (44.5, 29.2), turned to 180 degrees
- moved R27 47.0 mm to (49.5, 23.5)
- moved Q5 46.9 mm to (39.4, 17.1)
- moved Q6 46.9 mm to (44.5, 17.1)
- moved R21 46.9 mm to (43.8, 14.0)
- moved R22 46.9 mm to (39.4, 14.0)
- moved C21 37.0 mm to (68.6, 47.0), turned to 0 degrees
- moved U7 36.1 mm to (69.8, 50.8), turned to 180 degrees
- moved LED8 35.4 mm to (88.9, 72.4), turned to 270 degrees
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Connections:
- net ADC_POTI_BIT_ERROR_RATE: now also U2.42; no longer U2.40
- net ADC_POTI_DROP_DURATION: now also U2.40; no longer U2.42
Routing:
- net GND: track 231.3 -> 449.6 mm, vias 2 -> 6
- net ADC_REF: track 9.49 -> 120.6 mm
- net VSS: track 11.4 -> 120.8 mm, vias 0 -> 5
- net !SIM_LO: track 8.37 -> 103.1 mm, vias 0 -> 1
- net UART_EXP_RX: track 3.06 -> 88.6 mm, vias 0 -> 2
- net !SIM_SOE: track 7.27 -> 90.8 mm
- net ADC_POTI_BIT_ERROR_RATE: track 0.00 -> 82.8 mm
- net UART_EXP_TX: track 3.98 -> 86.6 mm, vias 0 -> 2
- net ADC_CURRENT_SENSE: track 35.1 -> 112.6 mm, vias 0 -> 2
- net !SIM_SODS: track 12.0 -> 88.2 mm, vias 0 -> 2
- net +3V3: track 111.7 -> 187.2 mm, vias 0 -> 2
- net EXPPWR_EN: track 10.7 -> 80.2 mm, vias 0 -> 2
- net SW_ERRINH: track 2.56 -> 67.9 mm, vias 0 -> 2
- net VDD: track 25.9 -> 85.3 mm, vias 0 -> 2
- net DEBUG_TX_D+: track 0.00 -> 54.1 mm
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- added copper zone on layer 16, net VSS
