File: eagle/rxsms-2.0.sch (EAGLE design)
At the start: 160 parts, among them Q1 opt, Q10 BSS123, Q11 BSS123, Q12 BSS123, Q2 BSS123, Q3 BSS123, Q4 BSS123, Q5 BSS123, Q6 BSS123, Q7 BSS123, Q8 BSS123, Q9 BSS123, T10_SODS SWITCH_LED, T1_LO SMS_IP67, T2_SOE SMS_IP67, T3_SOE SWITCH_LED, T4_PWR SMS_IP67, T5_ERRINH SMS_IP67, T6_PWR SWITCH_LED, T7_ERRINH SWITCH_LED, T8_LO SWITCH_LED, T9_SODS SMS_IP67, U1 MAX3232ESE, U2 XMEGA-A4UTQFP, U3 TSR_1-2450, U4 LM1117, U5 NC7WZ17P6X, U6 ADUM3160, U7 TPS73125, U8 NUP2202W1, X1 PN61729-S, X5 RLP2-200-500

Commit message: continued layout
Parts:
- R21, R23, R24, R26, R27, R28, R30, R31: OC_FARNELL (none) -> 1887308
- U2: OC_FARNELL (none) -> 2066309
Changed lines of the file:
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@@
 <part name="VSS3" library="supply1" deviceset="VSS" device=""/>
 <part name="VSS4" library="supply1" deviceset="VSS" device=""/>
-<part name="U2" library="avr-7" deviceset="XMEGA-A4U" device="TQFP"/>
+<part name="U2" library="avr-7" deviceset="XMEGA-A4U" device="TQFP">
+<attribute name="OC_FARNELL" value="2066309"/>
+</part>
 <part name="FRAME1" library="frames" deviceset="DINA4_L" device=""/>
 <part name="C6" library="rcl" deviceset="C-EU" device="C0805K" value="100n"/>
@@
 <part name="Q6" library="transistor-small-signal" deviceset="BSS123" device=""/>
 <part name="GND23" library="supply1" deviceset="GND" device=""/>
-<part name="R21" library="rcl" deviceset="R-EU_" device="R0805" value="10k"/>
+<part name="R21" library="rcl" deviceset="R-EU_" device="R0805" value="10k">
+<attribute name="OC_FARNELL" value="1887308"/>
+</part>
 <part name="R22" library="rcl" deviceset="R-EU_" device="R0805" value="127"/>
 <part name="+3V8" library="supply1" deviceset="+3V3" device=""/>
 <part name="VDD3" library="supply1" deviceset="VDD" device=""/>
-<part name="R23" library="rcl" deviceset="R-EU_" device="R0805" value="10k"/>
+<part name="R23" library="rcl" deviceset="R-EU_" device="R0805" value="10k">
+<attribute name="OC_FARNELL" value="1887308"/>
+</part>
 <part name="VSS6" library="supply1" deviceset="VSS" device=""/>
 <part name="OK2" library="optocoupler" deviceset="HCPL0600" device=""/>
@@
 <part name="Q8" library="transistor-small-signal" deviceset="BSS123" device=""/>
 <part name="GND24" library="supply1" deviceset="GND" device=""/>
-<part name="R24" library="rcl" deviceset="R-EU_" device="R0805" value="10k"/>
+<part name="R24" library="rcl" deviceset="R-EU_" device="R0805" value="10k">
+<attribute name="OC_FARNELL" value="1887308"/>
+</part>
 <part name="R25" library="rcl" deviceset="R-EU_" device="R0805" value="127"/>
 <part name="+3V9" library="supply1" deviceset="+3V3" device=""/>
 <part name="VDD4" library="supply1" deviceset="VDD" device=""/>
-<part name="R26" library="rcl" deviceset="R-EU_" device="R0805" value="10k"/>
+<part name="R26" library="rcl" deviceset="R-EU_" device="R0805" value="10k">
+<attribute name="OC_FARNELL" value="1887308"/>
+</part>
 <part name="VSS7" library="supply1" deviceset="VSS" device=""/>
 <part name="OK3" library="optocoupler" deviceset="HCPL0600" device=""/>
-<part name="R27" library="rcl" deviceset="R-EU_" device="R0805" value="10k"/>
+<part name="R27" library="rcl" deviceset="R-EU_" device="R0805" value="10k">
+<attribute name="OC_FARNELL" value="1887308"/>
+</part>
 <part name="+3V10" library="supply1" deviceset="+3V3" device=""/>
 <part name="GND25" library="supply1" deviceset="GND" device=""/>
 <part name="Q9" library="transistor-small-signal" deviceset="BSS123" device=""/>
 <part name="Q10" library="transistor-small-signal" deviceset="BSS123" device=""/>
-<part name="R28" library="rcl" deviceset="R-EU_" device="R0805" value="10k"/>
+<part name="R28" library="rcl" deviceset="R-EU_" device="R0805" value="10k">
+<attribute name="OC_FARNELL" value="1887308"/>
+</part>
 <part name="R29" library="rcl" deviceset="R-EU_" device="R0805" value="267"/>
 <part name="VDD5" library="supply1" deviceset="VDD" device=""/>
 <part name="VSS8" library="supply1" deviceset="VSS" device=""/>
 <part name="OK4" library="optocoupler" deviceset="HCPL0600" device=""/>
-<part name="R30" library="rcl" deviceset="R-EU_" device="R0805" value="10k"/>
+<part name="R30" library="rcl" deviceset="R-EU_" device="R0805" value="10k">
+<attribute name="OC_FARNELL" value="1887308"/>
+</part>
 <part name="+3V11" library="supply1" deviceset="+3V3" device=""/>
 <part name="GND26" library="supply1" deviceset="GND" device=""/>
 <part name="Q11" library="transistor-small-signal" deviceset="BSS123" device=""/>
 <part name="Q12" library="transistor-small-signal" deviceset="BSS123" device=""/>
-<part name="R31" library="rcl" deviceset="R-EU_" device="R0805" value="10k"/>
+<part name="R31" library="rcl" deviceset="R-EU_" device="R0805" value="10k">
+<attribute name="OC_FARNELL" value="1887308"/>
+</part>
 <part name="R32" library="rcl" deviceset="R-EU_" device="R0805" value="267"/>
 <part name="VDD6" library="supply1" deviceset="VDD" device=""/>
@@
 </plain>
 <instances>
-<instance part="U2" gate="G$1" x="124.46" y="104.14"/>
+<instance part="U2" gate="G$1" x="124.46" y="104.14">
+<attribute name="OC_FARNELL" x="124.46" y="104.14" size="1.778" layer="96" display="off"/>
+</instance>
 <instance part="FRAME1" gate="G$1" x="0" y="0"/>
 <instance part="FRAME1" gate="G$2" x="162.56" y="0"/>
@@
 <instance part="Q6" gate="G$1" x="53.34" y="149.86"/>
 <instance part="GND23" gate="1" x="53.34" y="139.7"/>
-<instance part="R21" gate="G$1" x="53.34" y="160.02" rot="R90"/>
+<instance part="R21" gate="G$1" x="53.34" y="160.02" rot="R90">
+<attribute name="OC_FARNELL" x="53.34" y="160.02" size="1.778" layer="96" rot="R90" display="off"/>
+</instance>
 <instance part="R22" gate="G$1" x="71.12" y="160.02" rot="R90"/>
 <instance part="+3V8" gate="G$1" x="53.34" y="170.18"/>
 <instance part="VDD3" gate="G$1" x="104.14" y="167.64"/>
-<instance part="R23" gate="G$1" x="109.22" y="154.94" rot="R90"/>
+<instance part="R23" gate="G$1" x="109.22" y="154.94" rot="R90">
+<attribute name="OC_FARNELL" x="109.22" y="154.94" size="1.778" layer="96" rot="R90" display="off"/>
+</instance>
 <instance part="VSS6" gate="G$1" x="104.14" y="139.7"/>
 <instance part="OK2" gate="A" x="86.36" y="66.04"/>
@@
 <instance part="Q8" gate="G$1" x="53.34" y="68.58"/>
 <instance part="GND24" gate="1" x="53.34" y="58.42"/>
-<instance part="R24" gate="G$1" x="53.34" y="78.74" rot="R90"/>
+<instance part="R24" gate="G$1" x="53.34" y="78.74" rot="R90">
+<attribute name="OC_FARNELL" x="53.34" y="78.74" size="1.778" layer="96" rot="R90" display="off"/>
+</instance>
 <instance part="R25" gate="G$1" x="71.12" y="78.74" rot="R90"/>
 <instance part="+3V9" gate="G$1" x="53.34" y="88.9"/>
 <instance part="VDD4" gate="G$1" x="104.14" y="86.36"/>
-<instance part="R26" gate="G$1" x="109.22" y="73.66" rot="R90"/>
+<instance part="R26" gate="G$1" x="109.22" y="73.66" rot="R90">
+<attribute name="OC_FARNELL" x="109.22" y="73.66" size="1.778" layer="96" rot="R90" display="off"/>
+</instance>
 <instance part="VSS7" gate="G$1" x="104.14" y="58.42"/>
 <instance part="OK3" gate="A" x="86.36" y="106.68" rot="MR0"/>
-<instance part="R27" gate="G$1" x="63.5" y="114.3" rot="R90"/>
+<instance part="R27" gate="G$1" x="63.5" y="114.3" rot="R90">
+<attribute name="OC_FARNELL" x="63.5" y="114.3" size="1.778" layer="96" rot="R90" display="off"/>
+</instance>
 <instance part="+3V10" gate="G$1" x="68.58" y="127"/>
 <instance part="GND25" gate="1" x="68.58" y="99.06"/>
 <instance part="Q9" gate="G$1" x="104.14" y="104.14" rot="MR270"/>
 <instance part="Q10" gate="G$1" x="119.38" y="109.22" rot="MR0"/>
-<instance part="R28" gate="G$1" x="119.38" y="119.38" rot="R90"/>
+<instance part="R28" gate="G$1" x="119.38" y="119.38" rot="R90">
+<attribute name="OC_FARNELL" x="119.38" y="119.38" size="1.778" layer="96" rot="R90" display="off"/>
+</instance>
 <instance part="R29" gate="G$1" x="101.6" y="119.38" rot="R90"/>
 <instance part="VDD5" gate="G$1" x="101.6" y="129.54"/>
 <instance part="VSS8" gate="G$1" x="119.38" y="99.06"/>
 <instance part="OK4" gate="A" x="86.36" y="25.4" rot="MR0"/>
-<instance part="R30" gate="G$1" x="63.5" y="33.02" rot="R90"/>
+<instance part="R30" gate="G$1" x="63.5" y="33.02" rot="R90">
+<attribute name="OC_FARNELL" x="63.5" y="33.02" size="1.778" layer="96" rot="R90" display="off"/>
+</instance>
 <instance part="+3V11" gate="G$1" x="68.58" y="45.72"/>
 <instance part="GND26" gate="1" x="68.58" y="17.78"/>
 <instance part="Q11" gate="G$1" x="104.14" y="22.86" rot="MR270"/>
 <instance part="Q12" gate="G$1" x="119.38" y="27.94" rot="MR0"/>
-<instance part="R31" gate="G$1" x="119.38" y="38.1" rot="R90"/>
+<instance part="R31" gate="G$1" x="119.38" y="38.1" rot="R90">
+<attribute name="OC_FARNELL" x="119.38" y="38.1" size="1.778" layer="96" rot="R90" display="off"/>
+</instance>
 <instance part="R32" gate="G$1" x="101.6" y="38.1" rot="R90"/>
 <instance part="VDD6" gate="G$1" x="101.6" y="48.26"/>

Commit message: more OC_FARNELL added
Parts:
- R1, R10, R11, R2, R3, R5, R6, R8, R9: OC_FARNELL (none) -> 1887308
- R7: OC_FARNELL (none) -> 2333538
Changed lines of the file:
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@@
 <part name="VDD2" library="supply1" deviceset="VDD" device=""/>
 <part name="VSS5" library="supply1" deviceset="VSS" device=""/>
-<part name="R1" library="rcl" deviceset="R-EU_" device="R0805" value="10k"/>
+<part name="R1" library="rcl" deviceset="R-EU_" device="R0805" value="10k">
+<attribute name="OC_FARNELL" value="1887308"/>
+</part>
 <part name="FRAME4" library="frames" deviceset="DINA4_L" device=""/>
 <part name="X4" library="con-subd" deviceset="F15HP" device=""/>
@@
 <part name="Q2" library="transistor-small-signal" deviceset="BSS123" device=""/>
 <part name="U$5" library="SP491" deviceset="SP490" device=""/>
-<part name="R2" library="rcl" deviceset="R-EU_" device="R0805" value="10k"/>
+<part name="R2" library="rcl" deviceset="R-EU_" device="R0805" value="10k">
+<attribute name="OC_FARNELL" value="1887308"/>
+</part>
 <part name="GND8" library="supply1" deviceset="GND" device=""/>
 <part name="+3V4" library="supply1" deviceset="+3V3" device=""/>
-<part name="R3" library="rcl" deviceset="R-EU_" device="R0805" value="10k"/>
+<part name="R3" library="rcl" deviceset="R-EU_" device="R0805" value="10k">
+<attribute name="OC_FARNELL" value="1887308"/>
+</part>
 <part name="R4" library="rcl" deviceset="R-EU_" device="R0805" value="22k"/>
 <part name="U$6" library="BTS6134" deviceset="BTS6143" device=""/>
 <part name="P+1" library="supply1" deviceset="+24V" device="" value="+28V_SUPPLY"/>
-<part name="R5" library="rcl" deviceset="R-EU_" device="R0805" value="10k"/>
+<part name="R5" library="rcl" deviceset="R-EU_" device="R0805" value="10k">
+<attribute name="OC_FARNELL" value="1887308"/>
+</part>
 <part name="GND9" library="supply1" deviceset="GND" device=""/>
-<part name="R6" library="rcl" deviceset="R-EU_" device="R0805" value="10k"/>
-<part name="R7" library="rcl" deviceset="R-EU_" device="R0805" value="100k"/>
+<part name="R6" library="rcl" deviceset="R-EU_" device="R0805" value="10k">
+<attribute name="OC_FARNELL" value="1887308"/>
+</part>
+<part name="R7" library="rcl" deviceset="R-EU_" device="R0805" value="100k">
+<attribute name="OC_FARNELL" value="2333538"/>
+</part>
 <part name="C16" library="rcl" deviceset="C-EU" device="C0805K" value="100n"/>
 <part name="Q3" library="transistor-small-signal" deviceset="BSS123" device=""/>
-<part name="R8" library="rcl" deviceset="R-EU_" device="R0805" value="10k"/>
-<part name="R9" library="rcl" deviceset="R-EU_" device="R0805" value="10k"/>
+<part name="R8" library="rcl" deviceset="R-EU_" device="R0805" value="10k">
+<attribute name="OC_FARNELL" value="1887308"/>
+</part>
+<part name="R9" library="rcl" deviceset="R-EU_" device="R0805" value="10k">
+<attribute name="OC_FARNELL" value="1887308"/>
+</part>
 <part name="P+5" library="supply1" deviceset="+5V" device=""/>
 <part name="P+6" library="supply1" deviceset="+5V" device=""/>
@@
 <part name="+3V5" library="supply1" deviceset="+3V3" device=""/>
 <part name="Q4" library="transistor-small-signal" deviceset="BSS123" device=""/>
-<part name="R10" library="rcl" deviceset="R-EU_" device="R0805" value="10k"/>
-<part name="R11" library="rcl" deviceset="R-EU_" device="R0805" value="10k"/>
+<part name="R10" library="rcl" deviceset="R-EU_" device="R0805" value="10k">
+<attribute name="OC_FARNELL" value="1887308"/>
+</part>
+<part name="R11" library="rcl" deviceset="R-EU_" device="R0805" value="10k">
+<attribute name="OC_FARNELL" value="1887308"/>
+</part>
 <part name="P+7" library="supply1" deviceset="+5V" device=""/>
 <part name="+3V6" library="supply1" deviceset="+3V3" device=""/>
@@
 <instance part="+3V2" gate="G$1" x="15.24" y="88.9"/>
 <instance part="GND3" gate="1" x="15.24" y="63.5"/>
-<instance part="R1" gate="G$1" x="30.48" y="83.82"/>
+<instance part="R1" gate="G$1" x="30.48" y="83.82">
+<attribute name="OC_FARNELL" x="30.48" y="83.82" size="1.778" layer="96" display="off"/>
+</instance>
 <instance part="+3V14" gate="G$1" x="40.64" y="53.34" rot="MR0"/>
 <instance part="GND37" gate="1" x="218.44" y="101.6"/>
@@
 <instance part="Q2" gate="G$1" x="121.92" y="165.1"/>
 <instance part="U$5" gate="G$1" x="96.52" y="27.94"/>
-<instance part="R2" gate="G$1" x="142.24" y="96.52" rot="R90"/>
+<instance part="R2" gate="G$1" x="142.24" y="96.52" rot="R90">
+<attribute name="OC_FARNELL" x="142.24" y="96.52" size="1.778" layer="96" rot="R90" display="off"/>
+</instance>
 <instance part="GND8" gate="1" x="210.82" y="88.9" rot="R90"/>
 <instance part="+3V4" gate="G$1" x="175.26" y="109.22"/>
-<instance part="R3" gate="G$1" x="152.4" y="96.52" rot="R90"/>
+<instance part="R3" gate="G$1" x="152.4" y="96.52" rot="R90">
+<attribute name="OC_FARNELL" x="152.4" y="96.52" size="1.778" layer="96" rot="R90" display="off"/>
+</instance>
 <instance part="R4" gate="G$1" x="38.1" y="96.52" rot="R90"/>
 <instance part="U$6" gate="G$1" x="167.64" y="160.02"/>
 <instance part="P+1" gate="1" x="213.36" y="172.72" rot="R270"/>
-<instance part="R5" gate="G$1" x="111.76" y="149.86" rot="R90"/>
+<instance part="R5" gate="G$1" x="111.76" y="149.86" rot="R90">
+<attribute name="OC_FARNELL" x="111.76" y="149.86" size="1.778" layer="96" rot="R90" display="off"/>
+</instance>
 <instance part="GND9" gate="1" x="121.92" y="137.16"/>
-<instance part="R6" gate="G$1" x="121.92" y="40.64" rot="R90"/>
-<instance part="R7" gate="G$1" x="121.92" y="22.86" rot="R90"/>
+<instance part="R6" gate="G$1" x="121.92" y="40.64" rot="R90">
+<attribute name="OC_FARNELL" x="121.92" y="40.64" size="1.778" layer="96" rot="R90" display="off"/>
+</instance>
+<instance part="R7" gate="G$1" x="121.92" y="22.86" rot="R90">
+<attribute name="OC_FARNELL" x="121.92" y="22.86" size="1.778" layer="96" rot="R90" display="off"/>
+</instance>
 <instance part="C16" gate="G$1" x="60.96" y="33.02"/>
 <instance part="Q3" gate="G$1" x="38.1" y="45.72" rot="R270"/>
-<instance part="R8" gate="G$1" x="27.94" y="50.8" rot="R90"/>
-<instance part="R9" gate="G$1" x="45.72" y="50.8" rot="R90"/>
+<instance part="R8" gate="G$1" x="27.94" y="50.8" rot="R90">
+<attribute name="OC_FARNELL" x="27.94" y="50.8" size="1.778" layer="96" rot="R90" display="off"/>
+</instance>
+<instance part="R9" gate="G$1" x="45.72" y="50.8" rot="R90">
+<attribute name="OC_FARNELL" x="45.72" y="50.8" size="1.778" layer="96" rot="R90" display="off"/>
+</instance>
 <instance part="P+5" gate="1" x="45.72" y="60.96"/>
 <instance part="P+6" gate="1" x="60.96" y="43.18"/>
@@
 <instance part="+3V5" gate="G$1" x="27.94" y="60.96"/>
 <instance part="Q4" gate="G$1" x="38.1" y="12.7" rot="R270"/>
-<instance part="R10" gate="G$1" x="27.94" y="17.78" rot="R90"/>
-<instance part="R11" gate="G$1" x="45.72" y="17.78" rot="R90"/>
+<instance part="R10" gate="G$1" x="27.94" y="17.78" rot="R90">
+<attribute name="OC_FARNELL" x="27.94" y="17.78" size="1.778" layer="96" rot="R90" display="off"/>
+</instance>
+<instance part="R11" gate="G$1" x="45.72" y="17.78" rot="R90">
+<attribute name="OC_FARNELL" x="45.72" y="17.78" size="1.778" layer="96" rot="R90" display="off"/>
+</instance>
 <instance part="P+7" gate="1" x="45.72" y="27.94"/>
 <instance part="+3V6" gate="G$1" x="27.94" y="27.94"/>

Commit message: fix: use correct lib name for TEN 3-2410N DCDC iso regulator
Parts:
- U$10: value TES3-4810WI -> TEN3-2410N; device TES3-4810WI:TES3-4810WI -> TEN3:TEN3-2410N
- U3: OC_FARNELL (none) -> 1696320
Changed lines of the file:
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@@
 <part name="GND3" library="supply1" deviceset="GND" device=""/>
 <part name="FRAME3" library="frames" deviceset="DINA4_L" device=""/>
-<part name="U3" library="_traco_tsr-1" deviceset="TSR_1-*" device="" technology="2450"/>
+<part name="U3" library="_traco_tsr-1" deviceset="TSR_1-*" device="" technology="2450">
+<attribute name="OC_FARNELL" value="1696320"/>
+</part>
 <part name="C12" library="rcl" deviceset="C-EU" device="C0805K" value="4u7/50V"/>
 <part name="C13" library="rcl" deviceset="C-EU" device="C0805K" value="4u7/50V"/>
@@
 <part name="P+15" library="supply1" deviceset="+24V" device="" value="+28V_SUPPLY"/>
 <part name="GND40" library="supply1" deviceset="GND" device=""/>
-<part name="U$10" library="TES3-4810WI" deviceset="TES3-4810WI" device=""/>
+<part name="U$10" library="TEN3" deviceset="TEN3-2410N" device=""/>
 <part name="C30" library="rcl" deviceset="C-EU" device="C0805K" value="4u7/50V"/>
 <part name="P+4" library="supply1" deviceset="+24V" device="" value="+28V_SUPPLY"/>
