File: eagle/rxsms-2.0.sch (EAGLE design)
At the start: 160 parts, among them Q1 opt, Q10 BSS123, Q11 BSS123, Q12 BSS123, Q2 BSS123, Q3 BSS123, Q4 BSS123, Q5 BSS123, Q6 BSS123, Q7 BSS123, Q8 BSS123, Q9 BSS123, T10_SODS SWITCH_LED, T1_LO SMS_IP67, T2_SOE SMS_IP67, T3_SOE SWITCH_LED, T4_PWR SMS_IP67, T5_ERRINH SMS_IP67, T6_PWR SWITCH_LED, T7_ERRINH SWITCH_LED, T8_LO SWITCH_LED, T9_SODS SMS_IP67, U1 MAX3232ESE, U2 XMEGA-A4UTQFP, U3 TSR_1-2450, U4 LM1117, U5 NC7WZ17P6X, U6 ADUM3160, U7 TPS73125, U8 NUP2202W1, X1 PN61729-S, X5 RLP2-200-500

Commit message: more OC added
Parts:
- C32: device rcl:C-EUC1206K -> rcl:C-EUC0805K
- C34: OC_FARNELL (none) -> 1759241
- D1: OC_FARNELL (none) -> 1081418
- R12, R13, R14, R15: OC_FARNELL (none) -> 1894163
- R4: OC_FARNELL (none) -> 2303686
- R48: OC_FARNELL (none) -> 2332111
- U$6: OC_FARNELL (none) -> 1440813
- U6: OC_FARNELL (none) -> 1843660
- U7: OC_FARNELL (none) -> 2112625
- X1: OC_FARNELL (none) -> 1642035
Changed lines of the file:
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@@
 <attribute name="OC_FARNELL" value="1887308"/>
 </part>
-<part name="R4" library="rcl" deviceset="R-EU_" device="R0805" value="22k"/>
-<part name="U$6" library="BTS6134" deviceset="BTS6143" device=""/>
+<part name="R4" library="rcl" deviceset="R-EU_" device="R0805" value="22k">
+<attribute name="OC_FARNELL" value="2303686"/>
+</part>
+<part name="U$6" library="BTS6134" deviceset="BTS6143" device="">
+<attribute name="OC_FARNELL" value="1440813"/>
+</part>
 <part name="P+1" library="supply1" deviceset="+24V" device="" value="+28V_SUPPLY"/>
 <part name="R5" library="rcl" deviceset="R-EU_" device="R0805" value="10k">
@@
 <part name="+3V6" library="supply1" deviceset="+3V3" device=""/>
 <part name="GND10" library="supply1" deviceset="GND" device=""/>
-<part name="U6" library="adum3160" deviceset="ADUM3160" device=""/>
+<part name="U6" library="adum3160" deviceset="ADUM3160" device="">
+<attribute name="OC_FARNELL" value="1843660"/>
+</part>
 <part name="FRAME5" library="frames" deviceset="DINA4_L" device=""/>
 <part name="C17" library="rcl" deviceset="C-EU" device="C0805K" value="&gt;100n/low ESR"/>
-<part name="R12" library="rcl" deviceset="R-EU_" device="R0805" value="24/1%"/>
+<part name="R12" library="rcl" deviceset="R-EU_" device="R0805" value="24/1%">
+<attribute name="OC_FARNELL" value="1894163"/>
+</part>
 <part name="GND12" library="supply1" deviceset="GND" device=""/>
 <part name="+3V7" library="supply1" deviceset="+3V3" device=""/>
 <part name="C18" library="rcl" deviceset="C-EU" device="C0805K" value="&gt;100n/low ESR"/>
-<part name="R13" library="rcl" deviceset="R-EU_" device="R0805" value="24/1%"/>
+<part name="R13" library="rcl" deviceset="R-EU_" device="R0805" value="24/1%">
+<attribute name="OC_FARNELL" value="1894163"/>
+</part>
 <part name="C19" library="rcl" deviceset="C-EU" device="C0805K" value="&gt;100n/low ESR"/>
 <part name="C20" library="rcl" deviceset="C-EU" device="C0805K" value="&gt;100n/low ESR"/>
-<part name="R14" library="rcl" deviceset="R-EU_" device="R0805" value="24/1%"/>
-<part name="R15" library="rcl" deviceset="R-EU_" device="R0805" value="24/1%"/>
+<part name="R14" library="rcl" deviceset="R-EU_" device="R0805" value="24/1%">
+<attribute name="OC_FARNELL" value="1894163"/>
+</part>
+<part name="R15" library="rcl" deviceset="R-EU_" device="R0805" value="24/1%">
+<attribute name="OC_FARNELL" value="1894163"/>
+</part>
 <part name="U4" library="LM1117" deviceset="LM1117" device=""/>
 <part name="P+8" library="supply1" deviceset="+12V" device="" value="+28V_EXP"/>
 <part name="P+9" library="supply1" deviceset="+12V" device="" value="+28V_EXP"/>
 <part name="P+10" library="supply1" deviceset="+12V" device="" value="+28V_EXP"/>
-<part name="X1" library="con-berg" deviceset="PN61729-S" device=""/>
+<part name="X1" library="con-berg" deviceset="PN61729-S" device="">
+<attribute name="OC_FARNELL" value="1642035"/>
+</part>
 <part name="FRAME6" library="frames" deviceset="DINA4_L" device=""/>
-<part name="U7" library="TPS731xx" deviceset="TPS731*" device="" value="TPS73125"/>
+<part name="U7" library="TPS731xx" deviceset="TPS731*" device="" value="TPS73125">
+<attribute name="OC_FARNELL" value="2112625"/>
+</part>
 <part name="U$7_BER" library="poti" deviceset="STRK11K" device=""/>
 <part name="P+11" library="supply1" deviceset="+5V" device=""/>
@@
 <part name="C29" library="rcl" deviceset="C-EU" device="C0805K" value="100n"/>
 <part name="GND21" library="supply1" deviceset="GND" device=""/>
-<part name="C32" library="rcl" deviceset="C-EU" device="C1206K" value="10u/16V"/>
+<part name="C32" library="rcl" deviceset="C-EU" device="C0805K" value="10u/16V"/>
 <part name="C33" library="rcl" deviceset="C-EU" device="C0805K" value="100n"/>
 <part name="GND22" library="supply1" deviceset="GND" device=""/>
@@
 <part name="GND33" library="supply1" deviceset="GND" device=""/>
 <part name="U8" library="nup2202w1" deviceset="NUP2202W1" device=""/>
-<part name="C34" library="rcl" deviceset="C-EU" device="C0805K" value="4n7"/>
-<part name="R48" library="rcl" deviceset="R-EU_" device="R0805" value="1M"/>
+<part name="C34" library="rcl" deviceset="C-EU" device="C0805K" value="4n7">
+<attribute name="OC_FARNELL" value="1759241"/>
+</part>
+<part name="R48" library="rcl" deviceset="R-EU_" device="R0805" value="1M">
+<attribute name="OC_FARNELL" value="2332111"/>
+</part>
 <part name="LED7" library="led" deviceset="LED" device="CHIPLED_1206" value="BERNSTEIN">
 <attribute name="OC_FARNELL" value="2322083"/>
@@
 <part name="C39" library="rcl" deviceset="C-EU" device="C0805K" value="100n"/>
 <part name="GND41" library="supply1" deviceset="GND" device=""/>
-<part name="D1" library="diode" deviceset="ZENER-DIODE" device="SOT23" value="3V"/>
+<part name="D1" library="diode" deviceset="ZENER-DIODE" device="SOT23" value="3V">
+<attribute name="OC_FARNELL" value="1081418"/>
+</part>
 <part name="GND42" library="supply1" deviceset="GND" device=""/>
 <part name="U5" library="NC7WZ17" deviceset="NC7WZ17P6X" device=""/>
@@
 <instance part="FRAME3" gate="G$1" x="2.54" y="-2.54"/>
 <instance part="FRAME3" gate="G$2" x="165.1" y="-2.54"/>
-<instance part="U3" gate="G$1" x="78.74" y="124.46"/>
+<instance part="U3" gate="G$1" x="78.74" y="124.46">
+<attribute name="OC_FARNELL" x="78.74" y="124.46" size="1.778" layer="96" display="off"/>
+</instance>
 <instance part="C12" gate="G$1" x="35.56" y="116.84"/>
 <instance part="C13" gate="G$1" x="93.98" y="116.84"/>
@@
 <attribute name="OC_FARNELL" x="152.4" y="96.52" size="1.778" layer="96" rot="R90" display="off"/>
 </instance>
-<instance part="R4" gate="G$1" x="38.1" y="96.52" rot="R90"/>
-<instance part="U$6" gate="G$1" x="167.64" y="160.02"/>
+<instance part="R4" gate="G$1" x="38.1" y="96.52" rot="R90">
+<attribute name="OC_FARNELL" x="38.1" y="96.52" size="1.778" layer="96" rot="R90" display="off"/>
+</instance>
+<instance part="U$6" gate="G$1" x="167.64" y="160.02">
+<attribute name="OC_FARNELL" x="167.64" y="160.02" size="1.778" layer="96" display="off"/>
+</instance>
 <instance part="P+1" gate="1" x="213.36" y="172.72" rot="R270"/>
 <instance part="R5" gate="G$1" x="111.76" y="149.86" rot="R90">
@@
 <instance part="SJ3" gate="1" x="210.82" y="114.3"/>
 <instance part="R50" gate="G$1" x="134.62" y="149.86" rot="R90"/>
-<instance part="D1" gate="G$1" x="38.1" y="83.82" rot="R90"/>
+<instance part="D1" gate="G$1" x="38.1" y="83.82" rot="R90">
+<attribute name="OC_FARNELL" x="38.1" y="83.82" size="1.778" layer="96" rot="R90" display="off"/>
+</instance>
 <instance part="GND42" gate="1" x="38.1" y="73.66"/>
 <instance part="U5" gate="A" x="73.66" y="91.44"/>
@@
 </plain>
 <instances>
-<instance part="U6" gate="G$1" x="33.02" y="58.42" rot="MR0"/>
+<instance part="U6" gate="G$1" x="33.02" y="58.42" rot="MR0">
+<attribute name="OC_FARNELL" x="33.02" y="58.42" size="1.778" layer="96" rot="MR0" display="off"/>
+</instance>
 <instance part="FRAME5" gate="G$1" x="-93.98" y="-27.94"/>
 <instance part="FRAME5" gate="G$2" x="68.58" y="-27.94"/>
 <instance part="C17" gate="G$1" x="58.42" y="76.2"/>
-<instance part="R12" gate="G$1" x="76.2" y="66.04"/>
+<instance part="R12" gate="G$1" x="76.2" y="66.04">
+<attribute name="OC_FARNELL" x="76.2" y="66.04" size="1.778" layer="96" display="off"/>
+</instance>
 <instance part="GND12" gate="1" x="-7.62" y="48.26"/>
 <instance part="+3V7" gate="G$1" x="-7.62" y="86.36"/>
 <instance part="C18" gate="G$1" x="68.58" y="76.2"/>
-<instance part="R13" gate="G$1" x="76.2" y="58.42"/>
+<instance part="R13" gate="G$1" x="76.2" y="58.42">
+<attribute name="OC_FARNELL" x="76.2" y="58.42" size="1.778" layer="96" display="off"/>
+</instance>
 <instance part="C19" gate="G$1" x="2.54" y="76.2"/>
 <instance part="C20" gate="G$1" x="-7.62" y="76.2"/>
-<instance part="R14" gate="G$1" x="-15.24" y="66.04"/>
-<instance part="R15" gate="G$1" x="-15.24" y="58.42"/>
+<instance part="R14" gate="G$1" x="-15.24" y="66.04">
+<attribute name="OC_FARNELL" x="-15.24" y="66.04" size="1.778" layer="96" display="off"/>
+</instance>
+<instance part="R15" gate="G$1" x="-15.24" y="58.42">
+<attribute name="OC_FARNELL" x="-15.24" y="58.42" size="1.778" layer="96" display="off"/>
+</instance>
 <instance part="X1" gate="G$1" x="132.08" y="76.2"/>
 <instance part="U8" gate="G$1" x="99.06" y="40.64" rot="MR0"/>
-<instance part="C34" gate="G$1" x="116.84" y="66.04"/>
-<instance part="R48" gate="G$1" x="109.22" y="66.04" rot="R90"/>
+<instance part="C34" gate="G$1" x="116.84" y="66.04">
+<attribute name="OC_FARNELL" x="116.84" y="66.04" size="1.778" layer="96" display="off"/>
+</instance>
+<instance part="R48" gate="G$1" x="109.22" y="66.04" rot="R90">
+<attribute name="OC_FARNELL" x="109.22" y="66.04" size="1.778" layer="96" rot="R90" display="off"/>
+</instance>
 <instance part="SJ4" gate="1" x="124.46" y="66.04" rot="R270"/>
 </instances>
@@
 <instance part="FRAME6" gate="G$1" x="0" y="0"/>
 <instance part="FRAME6" gate="G$2" x="162.56" y="0"/>
-<instance part="U7" gate="G$1" x="25.4" y="160.02"/>
+<instance part="U7" gate="G$1" x="25.4" y="160.02">
+<attribute name="OC_FARNELL" x="25.4" y="160.02" size="1.778" layer="96" display="off"/>
+</instance>
 <instance part="U$7_BER" gate="G$1" x="71.12" y="147.32"/>
 <instance part="P+11" gate="1" x="7.62" y="167.64"/>

Commit message: more OC added
Parts:
- Q10, Q11, Q12, Q2, Q3, Q4, Q5, Q6, Q7, Q8, Q9: OC_FARNELL (none) -> 9558640RL; OC_RS (none) -> 545-0135
- SV1: OC_FARNELL (none) -> 1096983
- SV2, SV3, SV4, SV5, SV6: OC_FARNELL (none) -> 1096984; OC_RS (none) -> 740-7105
- U4: OC_FARNELL (none) -> 1685603
- U8: OC_RS (none) -> 463-690

Commit message: added even more OC
Parts:
- C1, C2, C3, C4, C5: OC_FARNELL (none) -> 2320853
- C12, C13, C30, C31, C35: OC_FARNELL (none) -> 2210979
- C14, C15: OC_FARNELL (none) -> 2346925
- C16, C21, C22, C23, C24, C25, C26, C27, C28, C29, C33, C36, C37, C38, C39, C40, C6, C7, C8, C9: OC_FARNELL (none) -> 1759265
- C17, C18, C19, C20: value >100n/low ESR -> 1u; OC_FARNELL (none) -> 2320853
- C32: OC_FARNELL (none) -> 2320856
- LED1_LO, LED2_SOE, LED3_SODS: OC_FARNELL (none) -> 2099249
- LED4_ERRINH, LED5_PWR, LED8: OC_FARNELL (none) -> 2099244
- R16, R17, R18, R19, R20: OC_FARNELL (none) -> 9237496
- R22, R25: OC_FARNELL (none) -> 2141745
- R29, R32: value 267 -> 270; OC_FARNELL (none) -> 2008375; OC_RS (none) -> 740-9019
- R36, R37, R38, R39, R40, R41, R42, R45, R46, R47: OC_FARNELL (none) -> 2074509
- R43, R44: value 220 -> 68; OC_FARNELL (none) -> 2074509
- R49: value 220 -> 150; OC_FARNELL (none) -> 1099794
- R50: OC_FARNELL (none) -> 1500705
- T10_SODS, T3_SOE, T8_LO: OC_BUERKLIN (none) -> 12 G 203
- T1_LO, T2_SOE, T4_PWR, T5_ERRINH, T9_SODS: OC_FARNELL (none) -> 1217758
- T6_PWR, T7_ERRINH: OC_BUERKLIN (none) -> 12 G 205
- U$4: OC_FARNELL (none) -> 1103848
- U$5: OC_FARNELL (none) -> 9387234
- U$7_BER, U$8_DROPR, U$9_DROPDUR: value (none) -> 50k; OC_FARNELL (none) -> 1345093
- X1: OC_RS (none) -> 515-1989
- X2_GROUNDSTATION, X3_DEBUG: OC_FARNELL (none) -> 1207597 (+2x 1855027)
- X4: OC_FARNELL (none) -> 1207598 (+2x 1855027)
Connections:
- net GND: now also U5.A2

Commit message: more finalization on the layout
Parts:
- X6: OC_FARNELL (none) -> 1131855
Changed lines of the file:
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@@
 <part name="GND39" library="supply1" deviceset="GND" device=""/>
 <part name="P+14" library="supply1" deviceset="+24V" device="" value="+28V_SUPPLY"/>
-<part name="X6" library="con-ptr500" deviceset="AK500/2" device=""/>
+<part name="X6" library="con-ptr500" deviceset="AK500/2" device="">
+<attribute name="OC_FARNELL" value="1131855"/>
+</part>
 <part name="P+15" library="supply1" deviceset="+24V" device="" value="+28V_SUPPLY"/>
 <part name="GND40" library="supply1" deviceset="GND" device=""/>
