File: eagle/rxsms-2.0-Stromvers.brd (EAGLE design)
At the start: 100 x 120.5 mm, 17 parts, among them Q1 FDD4141TO252

Commit message: Added logos, added ordering codes, otherwise minor changes
Routing:
- net GND: track 99.7 -> 97.8 mm
