File: eagle/rxsms-2.0-Stromvers.brd (EAGLE design)
At the start: 100 x 120.5 mm, 17 parts, among them Q1 FDD4141TO252

Commit message: fix schematics and layout
  o add a dummy package (circle) to the screw. without package, it does not
    appear in the BOM
  o update the order code for the screw: new model is a bit longer but
    much cheaper which is important because of the high number of pieces.
  o synchronize/update the screws in the layout files
Parts:
- added SCREW1, SCREW2: 4-40/M3, dsub-mounting-screw:SCREW_DUMMY
Changed lines of the file:
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@@
 <element name="SJ2" library="jumper" package="SJ" value="" x="57.5" y="73.28"/>
 <element name="SJ3" library="jumper" package="SJ" value="" x="57.5" y="77.265"/>
+<element name="SCREW1" library="dsub-mounting-screw" package="SCREW_DUMMY" value="4-40/M3" x="-7.4267" y="80">
+<attribute name="OC_FARNELL" value="2135988" x="-7.4267" y="80" size="1.778" layer="27" display="off"/>
+</element>
+<element name="SCREW2" library="dsub-mounting-screw" package="SCREW_DUMMY" value="4-40/M3" x="-7.0937" y="114">
+<attribute name="OC_FARNELL" value="2135988" x="-7.0937" y="114" size="1.778" layer="27" display="off"/>
+</element>
 </elements>
 <signals>
