File: eagle/simulator/rxsms-2.0.sch (EAGLE design)
At the start: 170 parts, among them Q1 opt, Q10 BSS123, Q11 BSS123, Q12 BSS123, Q13 FDD4141TO252, Q2 BSS123, Q3 BSS123, Q4 BSS123, Q5 BSS123, Q6 BSS123, Q7 BSS123, Q8 BSS123, Q9 BSS123, T10_SODS SWITCH_LED, T1_LO SMS_IP67, T2_SOE SMS_IP67, T3_SOE SWITCH_LED, T4_PWR SMS_IP67, T5_ERRINH SMS_IP67, T6_PWR SWITCH_LED, T7_ERRINH SWITCH_LED, T8_LO SWITCH_LED, T9_SODS SMS_IP67, U1 MAX3232ESE, U2 XMEGA-A4UTQFP, U3 TSR_1-2450, U4 LM1117, U5 NC7WZ17P6X, U6 ADUM3160, U7 TPS73125, U8 NUP2202W1, X1 PN61729-S, X5 RLP2-200-500

Commit message: changed OC of BSS123 FETs, use normal tape instead of re-reel'ed version
Parts:
- Q10, Q11, Q12, Q2, Q3, Q4, Q5, Q6, Q7, Q8, Q9: OC_FARNELL 9558640RL -> 9558640
Changed lines of the file:
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@@
 </part>
 <part name="Q2" library="transistor-small-signal" deviceset="BSS123" device="">
-<attribute name="OC_FARNELL" value="9558640RL"/>
+<attribute name="OC_FARNELL" value="9558640"/>
 <attribute name="OC_RS" value="545-0135"/>
 </part>
@@
 </part>
 <part name="Q3" library="transistor-small-signal" deviceset="BSS123" device="">
-<attribute name="OC_FARNELL" value="9558640RL"/>
+<attribute name="OC_FARNELL" value="9558640"/>
 <attribute name="OC_RS" value="545-0135"/>
 </part>
@@
 <part name="+3V5" library="supply1" deviceset="+3V3" device=""/>
 <part name="Q4" library="transistor-small-signal" deviceset="BSS123" device="">
-<attribute name="OC_FARNELL" value="9558640RL"/>
+<attribute name="OC_FARNELL" value="9558640"/>
 <attribute name="OC_RS" value="545-0135"/>
 </part>
@@
 <part name="OK1" library="optocoupler" deviceset="HCPL0600" device=""/>
 <part name="Q5" library="transistor-small-signal" deviceset="BSS123" device="">
-<attribute name="OC_FARNELL" value="9558640RL"/>
+<attribute name="OC_FARNELL" value="9558640"/>
 <attribute name="OC_RS" value="545-0135"/>
 </part>
 <part name="Q6" library="transistor-small-signal" deviceset="BSS123" device="">
-<attribute name="OC_FARNELL" value="9558640RL"/>
+<attribute name="OC_FARNELL" value="9558640"/>
 <attribute name="OC_RS" value="545-0135"/>
 </part>
@@
 <part name="OK2" library="optocoupler" deviceset="HCPL0600" device=""/>
 <part name="Q7" library="transistor-small-signal" deviceset="BSS123" device="">
-<attribute name="OC_FARNELL" value="9558640RL"/>
+<attribute name="OC_FARNELL" value="9558640"/>
 <attribute name="OC_RS" value="545-0135"/>
 </part>
 <part name="Q8" library="transistor-small-signal" deviceset="BSS123" device="">
-<attribute name="OC_FARNELL" value="9558640RL"/>
+<attribute name="OC_FARNELL" value="9558640"/>
 <attribute name="OC_RS" value="545-0135"/>
 </part>
@@
 <part name="GND25" library="supply1" deviceset="GND" device=""/>
 <part name="Q9" library="transistor-small-signal" deviceset="BSS123" device="">
-<attribute name="OC_FARNELL" value="9558640RL"/>
+<attribute name="OC_FARNELL" value="9558640"/>
 <attribute name="OC_RS" value="545-0135"/>
 </part>
 <part name="Q10" library="transistor-small-signal" deviceset="BSS123" device="">
-<attribute name="OC_FARNELL" value="9558640RL"/>
+<attribute name="OC_FARNELL" value="9558640"/>
 <attribute name="OC_RS" value="545-0135"/>
 </part>
@@
 <part name="GND26" library="supply1" deviceset="GND" device=""/>
 <part name="Q11" library="transistor-small-signal" deviceset="BSS123" device="">
-<attribute name="OC_FARNELL" value="9558640RL"/>
+<attribute name="OC_FARNELL" value="9558640"/>
 <attribute name="OC_RS" value="545-0135"/>
 </part>
 <part name="Q12" library="transistor-small-signal" deviceset="BSS123" device="">
-<attribute name="OC_FARNELL" value="9558640RL"/>
-<attribute name="OC_RS" value="545-0135"/>
-</part>
+<attribute name="OC_FARNELL" value="9558640"/>
+<attribute name="OC_RS" value="545-0135"/>
+</part>
