File: eagle/simulator/rxsms-2.0.sch (EAGLE design)
At the start: 170 parts, among them Q1 opt, Q10 BSS123, Q11 BSS123, Q12 BSS123, Q13 FDD4141TO252, Q2 BSS123, Q3 BSS123, Q4 BSS123, Q5 BSS123, Q6 BSS123, Q7 BSS123, Q8 BSS123, Q9 BSS123, T10_SODS SWITCH_LED, T1_LO SMS_IP67, T2_SOE SMS_IP67, T3_SOE SWITCH_LED, T4_PWR SMS_IP67, T5_ERRINH SMS_IP67, T6_PWR SWITCH_LED, T7_ERRINH SWITCH_LED, T8_LO SWITCH_LED, T9_SODS SMS_IP67, U1 MAX3232ESE, U2 XMEGA-A4UTQFP, U3 TSR_1-2450, U4 LM1117, U5 NC7WZ17P6X, U6 ADUM3160, U7 TPS73125, U8 NUP2202W1, X1 PN61729-S, X5 RLP2-200-500

Commit message: fix OC for USB resistors
Parts:
- R14, R15: OC_FARNELL 1894163 -> (none); OC_RS (none) -> 666-2386
Changed lines of the file:
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@@
 </part>
 <part name="R14" library="rcl" deviceset="R-EU_" device="R0805" value="24/1%">
-<attribute name="OC_FARNELL" value="1894163"/>
+<attribute name="OC_RS" value="666-2386"/>
 </part>
 <part name="R15" library="rcl" deviceset="R-EU_" device="R0805" value="24/1%">
-<attribute name="OC_FARNELL" value="1894163"/>
+<attribute name="OC_RS" value="666-2386"/>
 </part>
 <part name="U4" library="LM1117" deviceset="LM1117" device="">
@@
 </instance>
 <instance part="R14" gate="G$1" x="-15.24" y="66.04">
-<attribute name="OC_FARNELL" x="-15.24" y="66.04" size="1.778" layer="96" display="off"/>
+<attribute name="OC_RS" x="-15.24" y="66.04" size="1.778" layer="96" display="off"/>
 </instance>
 <instance part="R15" gate="G$1" x="-15.24" y="58.42">
-<attribute name="OC_FARNELL" x="-15.24" y="58.42" size="1.778" layer="96" display="off"/>
+<attribute name="OC_RS" x="-15.24" y="58.42" size="1.778" layer="96" display="off"/>
 </instance>
 <instance part="X1" gate="G$1" x="132.08" y="76.2">

Commit message: make color and ordercode explicit for 4mm jacks
Parts:
- U$3: value JACK -> black; OC_FARNELL (none) -> 1854507
- U$9: value JACK -> red; OC_FARNELL (none) -> 1854508
Changed lines of the file:
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@@
 <part name="SJ6" library="jumper" deviceset="SJ" device=""/>
 <part name="P+16" library="supply1" deviceset="+24V" device="" value="+28V_SUPPLY"/>
-<part name="U$3" library="jack" deviceset="JACK" device=""/>
-<part name="U$9" library="jack" deviceset="JACK" device=""/>
+<part name="U$3" library="jack" deviceset="JACK" device="" value="black">
+<attribute name="OC_FARNELL" value="1854507"/>
+</part>
+<part name="U$9" library="jack" deviceset="JACK" device="" value="red">
+<attribute name="OC_FARNELL" value="1854508"/>
+</part>
 <part name="Q13" library="transistor-fet" deviceset="FDD4141" device="TO252">
 <attribute name="OC_FARNELL" value="2101406"/>
