File: eagle/simulator/rxsms-2.0.brd (EAGLE design)
At the start: 159 x 120.5 mm, 174 parts, among them Q1 opt, Q10 BSS123, Q11 BSS123, Q12 BSS123, Q13 FDD4141TO252, Q2 BSS123, Q3 BSS123, Q4 BSS123, Q5 BSS123, Q6 BSS123, Q7 BSS123, Q8 BSS123, Q9 BSS123, T10_SODS SWITCH_LED, T1_LO SMS_IP67, T2_SOE SMS_IP67, T3_SOE SWITCH_LED, T4_PWR SMS_IP67, T5_ERRINH SMS_IP67, T6_PWR SWITCH_LED, T7_ERRINH SWITCH_LED, T8_LO SWITCH_LED, T9_SODS SMS_IP67, U1 MAX3232ESE, U2 XMEGA-A4UTQFP, U3 TSR_1-2450, U4 LM1117, U5 NC7WZ17P6X, U6 ADUM3160, U7 TPS73125, U8 NUP2202W1, X1 PN61729-S, X5 RLP2-200-500

Commit message: make color and ordercode explicit for 4mm jacks
Parts:
- U$3: value JACK -> black
- U$9: value JACK -> red
Changed lines of the file:
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@@
 <element name="SJ5" library="jumper" package="SJ" value="" x="57.15" y="80.01"/>
 <element name="SJ6" library="jumper" package="SJ" value="" x="46.99" y="72.39" rot="R270"/>
-<element name="U$3" library="jack" package="JACK" value="JACK" x="124.46" y="104.14" rot="R270">
-<attribute name="OC_FARNELL" value="1854507 (black), 1854508 (red), 1854511 (blue), 1854510 (yellow)" x="124.46" y="104.14" size="1.778" layer="27" rot="R270" display="off"/>
+<element name="U$3" library="jack" package="JACK" value="black" x="124.46" y="104.14" rot="R270">
+<attribute name="OC_FARNELL" value="1854507" x="124.46" y="104.14" size="1.778" layer="27" rot="R270" display="off"/>
 </element>
-<element name="U$9" library="jack" package="JACK" value="JACK" x="109.22" y="104.14" rot="R270">
-<attribute name="OC_FARNELL" value="1854507 (black), 1854508 (red), 1854511 (blue), 1854510 (yellow)" x="109.22" y="104.14" size="1.778" layer="27" rot="R270" display="off"/>
+<element name="U$9" library="jack" package="JACK" value="red" x="109.22" y="104.14" rot="R270">
+<attribute name="OC_FARNELL" value="1854508" x="109.22" y="104.14" size="1.778" layer="27" rot="R270" display="off"/>
 </element>
 <element name="Q13" library="transistor-fet" package="TO252" value="FDD4141TO252" x="83.82" y="104.14" rot="R180">
