File: eagle/simulator/rxsms-2.0.brd (EAGLE design)
At the start: 159 x 120.5 mm, 174 parts, among them Q1 opt, Q10 BSS123, Q11 BSS123, Q12 BSS123, Q13 FDD4141TO252, Q2 BSS123, Q3 BSS123, Q4 BSS123, Q5 BSS123, Q6 BSS123, Q7 BSS123, Q8 BSS123, Q9 BSS123, T10_SODS SWITCH_LED, T1_LO SMS_IP67, T2_SOE SMS_IP67, T3_SOE SWITCH_LED, T4_PWR SMS_IP67, T5_ERRINH SMS_IP67, T6_PWR SWITCH_LED, T7_ERRINH SWITCH_LED, T8_LO SWITCH_LED, T9_SODS SMS_IP67, U1 MAX3232ESE, U2 XMEGA-A4UTQFP, U3 TSR_1-2450, U4 LM1117, U5 NC7WZ17P6X, U6 ADUM3160, U7 TPS73125, U8 NUP2202W1, X1 PN61729-S, X5 RLP2-200-500

Commit message: assing value to 0 Ohm resistors
Parts:
- R33, R34, R35: value opt -> 0
Changed lines of the file:
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@@
 <attribute name="OC_FARNELL" value="2332064" x="24.13" y="28.575" size="1.778" layer="27" rot="R90" display="off"/>
 </element>
-<element name="R33" library="rcl" package="R0805" value="opt" x="67.0306" y="11.9507" rot="R180">
+<element name="R33" library="rcl" package="R0805" value="0" x="67.0306" y="11.9507" rot="R180">
 <attribute name="OC_FARNELL" value="2309112" x="67.0306" y="11.9507" size="1.778" layer="27" rot="R180" display="off"/>
 </element>
-<element name="R34" library="rcl" package="R0805" value="opt" x="64.77" y="15.24" rot="R270">
+<element name="R34" library="rcl" package="R0805" value="0" x="64.77" y="15.24" rot="R270">
 <attribute name="OC_FARNELL" value="2309112" x="64.77" y="15.24" size="1.778" layer="27" rot="R270" display="off"/>
 </element>
-<element name="R35" library="rcl" package="R0805" value="opt" x="68.5548" y="14.0081" rot="R180">
+<element name="R35" library="rcl" package="R0805" value="0" x="68.5548" y="14.0081" rot="R180">
 <attribute name="OC_FARNELL" value="2309112" x="68.5548" y="14.0081" size="1.778" layer="27" rot="R180" display="off"/>
 </element>
